Commit message: Improvements to winch plugin + real rope vals

File: src/rr_robot_description/urdf/rope.xacro (robot description, xacro)
@@ -23,5 +23,5 @@
         <parent link="${winch_name_no_postfix}_${postfix}"/>
         <child link="rope_yaw_link_${postfix}"/>
-        <dynamics damping="0.5" />
+        <dynamics damping="1" />
       </joint>
       <!-- Rope pitch -->
@@ -37,5 +37,5 @@
           <parent link="rope_yaw_link_${postfix}"/>
           <child link="rope_pitch_link_${postfix}"/>
-          <dynamics damping="0.5" />
+          <dynamics damping="1" />
         </joint>
       <!-- rope prismatic joint (springed joint)-->

Commit message: added constant force to winch plugin

File: src/rr_robot_description/urdf/rope.xacro (robot description, xacro)
@@ -59,5 +59,5 @@
         <parent link="rope_pitch_link_${postfix}"/>
         <child link="rope_link_${postfix}" />
-        <dynamics damping="0.5" />
+        <dynamics damping="2" />
       </joint>
     </xacro:macro>
