Commit message: Added gravity to world, link world -> "dummy"

File: src/rr_robot_description/urdf/robot.urdf.xacro (robot description, xacro)
@@ -17,5 +17,6 @@
   <xacro:property name="arm_z_offset" value="0" />
   <!-- world base link -->
-  <link name="world">
+  <!-- If name="world" the robot wil be fixed in the world -->
+  <link name="dummy">
     <origin xyz="0 0 0" rpy="0 0 0"/>
   </link>
@@ -23,5 +24,5 @@
   <xacro:include filename="$(find rr_robot_description)/include/chassis/urdf/chassis.xacro" />
   <xacro:chassis_macro name="${robot_name}_chassis"
-                       parent_link="world"
+                       parent_link="dummy"
                        x_offset="-${arm_x_offset}"
                        y_offset="-${arm_y_offset}"

Commit message: first iter suspension done

File: src/rr_robot_description/urdf/robot.urdf.xacro (robot description, xacro)
@@ -99,4 +99,15 @@
                             z= "-0.11818"
                             postfix="te" />
+  <xacro:include filename="$(find rr_robot_description)/urdf/wheel_assembly/top_wheel.xacro" />
+  <xacro:top_wheel_macro parent="${robot_name}_chassis"
+                            x= "1.13039"
+                            y= "0.12962"
+                            z= "-0.1344"
+                            postfix="le" />
+  <xacro:top_wheel_macro parent="${robot_name}_chassis"
+                            x= "1.13039"
+                            y= "-0.12962"
+                            z= "-0.1344"
+                            postfix="te" />
   <!-- ******************************** Tranmissions ******************************** -->
   <xacro:include filename="$(find rr_robot_description)/urdf/transmissions.xacro" />

File: src/rr_robot_description/urdf/wheel_assembly/top_wheel.xacro (robot description, xacro)
@@ -18,5 +18,5 @@
         </link>
         <joint name="top_pivot_joint_${postfix}" type="revolute">
-            <origin xyz="${x+0.06343} ${y} ${z+0.01419}" rpy="0 0 0" />
+            <origin xyz="${x-0.10581} ${y-41} ${z-0.01217}" rpy="0 0 0" />
             <axis xyz="0 1 0" />
             <limit lower="${-range}" upper="${range}" effort="1000" velocity="1000"/>
@@ -32,6 +32,6 @@
         </link>
         <joint name="top_wheel_yaw_joint_${postfix}" type="revolute">
-            <origin xyz="1.13039 0.12962 -0.1344" rpy="0. 0. 1.5708" />
-            <axis rpy="0 0 0" xyz="0 0 1" />
+            <origin xyz="0.10581 0 0.01217" rpy="0. 0. 1.5708" />
+            <axis xyz="0 0 1" />
             <limit lower="-0.20" upper="0.20" effort="10000" velocity="1000" />
             <joint_properties damping="1.0" friction="1.0" />
@@ -62,5 +62,5 @@
           </link>
           <joint name="top_wheel_le_joint" type="continuous">
-            <origin xyz="1.13039 0.12962 -0.1344" rpy="0. 0. 1.5708" />
+            <origin xyz="0 41 0" />
             <axis rpy="0 0 0" xyz="0 1 0" />
             <parent link="yaw_link_${postfix}" />

Commit message: Working on suspension

File: src/rr_robot_description/urdf/robot.urdf.xacro (robot description, xacro)
@@ -94,4 +94,9 @@
                             z= "-0.11818"
                             postfix="le" />
+  <xacro:bottom_wheel_macro parent="${robot_name}_chassis"
+                            x= "-0.0251"
+                            y= "-0.1615"
+                            z= "-0.11818"
+                            postfix="te" />
   <!-- ******************************** Tranmissions ******************************** -->
   <xacro:include filename="$(find rr_robot_description)/urdf/transmissions.xacro" />

File: src/rr_robot_description/urdf/suspension.xacro (robot description, xacro)
@@ -3,42 +3,42 @@
     <xacro:macro name="suspension_macro" params="parent">
         <link name="rope_drive_te">
-            <inertial>
-              <mass value="1" />
-              <origin xyz="0 0 0" rpy="0 0 0" />
-              <inertia ixx="0.002526666666667" ixy="0" ixz="0" iyy="0.002526666666667" iyz="0" izz="0.005"/>
-            </inertial>
-            <visual>
-              <origin xyz="0 0 0" rpy="0 0 0" />
-              <geometry>
-                <mesh filename="package://rr_robot_description/include/chassis/meshes/RopeDrives/visual.STL" />
-              </geometry>
-              <material name="grey">
-                <color rgba="0.4 0.4 0.4 1" />
-              </material>
-            </visual>
-            <visual>
-              <origin rpy="${pi/2} 0 0" xyz="0.035 0 0" />
-              <geometry>
-                <box size="0.005 0.10 0.005" />
-              </geometry>
-              <material name="Grey">
-                <color rgba="0.6 0.6 0.6 1" />
-              </material>
-            </visual>
-            <collision>
-              <origin xyz="0 0 0" rpy="0 0 0" />
-              <geometry>
-                <mesh filename="package://rr_robot_description/include/chassis/meshes/RopeDrives/collision.STL" />
-              </geometry>
-            </collision>
-          </link>
-          <joint name="rope_drive_te_joint" type="continuous">
-            <origin xyz="0.92999 -0.24067 -0.0269" rpy="0.09857 0.09857 1.64405" />
-            <axis rpy="0 0 0" xyz="1 0 0" />
-            <limit effort="10000" velocity="1000" />
-            <joint_properties damping="1.0" friction="1.0" />
-            <parent link="${name}" />
-            <child link="rope_drive_te" />
-          </joint>
+          <inertial>
+            <mass value="1" />
+            <origin xyz="0 0 0" rpy="0 0 0" />
+            <inertia ixx="0.002526666666667" ixy="0" ixz="0" iyy="0.002526666666667" iyz="0" izz="0.005"/>
+          </inertial>
+          <visual>
+            <origin xyz="0 0 0" rpy="0 0 0" />
+            <geometry>
+              <mesh filename="package://rr_robot_description/include/chassis/meshes/RopeDrives/visual.STL" />
+            </geometry>
+            <material name="grey">
+              <color rgba="0.4 0.4 0.4 1" />
+            </material>
+          </visual>
+          <visual>
+            <origin rpy="${pi/2} 0 0" xyz="0.035 0 0" />
+            <geometry>
+              <box size="0.005 0.10 0.005" />
+            </geometry>
+            <material name="Grey">
+              <color rgba="0.6 0.6 0.6 1" />
+            </material>
+          </visual>
+          <collision>
+            <origin xyz="0 0 0" rpy="0 0 0" />
+            <geometry>
+              <mesh filename="package://rr_robot_description/include/chassis/meshes/RopeDrives/collision.STL" />
+            </geometry>
+          </collision>
+        </link>
+        <joint name="rope_drive_te_joint" type="continuous">
+          <origin xyz="0.92999 -0.24067 -0.0269" rpy="0.09857 0.09857 1.64405" />
+          <axis rpy="0 0 0" xyz="1 0 0" />
+          <limit effort="10000" velocity="1000" />
+          <joint_properties damping="1.0" friction="1.0" />
+          <parent link="${name}" />
+          <child link="rope_drive_te" />
+        </joint>
     </xacro:macro>
 </robot>

File: src/rr_robot_description/urdf/wheel_assembly/bottom_wheel.xacro (robot description, xacro)
@@ -1,4 +1,7 @@
 <?xml version="1.0"?>
-<robot xmlns:xacro="http://ros.org/wiki/xacro" name="suspension">
+<!-- because closed loops are not allowed in URDF, the suspension is simplified to a torsional spring
+    at the wheel mount revolute joint. This can approximate the more complicated suspension as long as
+    the range of motion is small -->
+<robot xmlns:xacro="http://ros.org/wiki/xacro" name="bot_wheel">
     <xacro:property name="range" value="0.174533" />
     <xacro:macro name="bottom_wheel_macro" params="parent x y z postfix">
@@ -15,8 +18,8 @@
             </visual>
         </link>
-        <joint name="bottom_wheel_mount_${postfix}_joint" type="revolute">
-            <origin xyz="${x+0.06343} 0 ${z+0.01419}" rpy="0 0 0" />
+        <joint name="bottom_pivot_joint_${postfix}" type="revolute">
+            <origin xyz="${x+0.06343} ${y} ${z+0.01419}" rpy="0 0 0" />
             <axis xyz="0 1 0" />
-            <limit lower="${range}" upper="${range}" effort="1000" velocity="1000"/>
+            <limit lower="${-range}" upper="${range}" effort="1000" velocity="1000"/>
             <parent link="${parent}" />
             <child link="bottom_wheel_mount_${postfix}"/>
@@ -25,63 +28,29 @@
         <link name="bottom_wheel_${postfix}">
             <inertial>
-                <mass value="0.001" />
+                <mass value="1" />
                 <inertia ixx="0.002526666666667" ixy="0" ixz="0" iyy="0.002526666666667" iyz="0" izz="0.005"/>
             </inertial>
             <visual>
-                <geometry>
-                    <box size="0.05 0.01 0.01"/>
-                </geometry>
+              <origin xyz="0 0 0" rpy="0 0 0" />
+              <geometry>
+                <mesh filename="package://rr_robot_description/include/chassis/meshes/BottomWheels/visual.STL" />
+              </geometry>
+              <material name="grey">
+                <color rgba="0.4 0.4 0.4 1" />
+              </material>
             </visual>
+            <collision>
+              <origin xyz="0 0 0" rpy="0 0 0" />
+              <geometry>
+                <mesh filename="package://rr_robot_description/include/chassis/meshes/BottomWheels/collision.STL" />
+              </geometry>
+            </collision>
         </link>
-        <joint name="bottom_wheel_${postfix}_joint" type="continuous">
-            <origin xyz="${x-0.06343} 0 ${z-0.01419}" rpy="0 0 0" />
+        <joint name="bottom_wheel_joint_${postfix}" type="continuous">
+            <origin xyz="-0.06343 0 -0.01419" rpy="0 0 0" />
             <axis xyz="0 1 0"/>
             <parent link="bottom_wheel_mount_${postfix}" />
             <child link="bottom_wheel_${postfix}" />
         </joint>
-    <!-- spring revolute joint link TODO: finish this -->
-    <!--TODO: finish this-->
-        <link name="pitch_link_${postfix}">
-            <inertial>
-                <mass value="0.001" />
-                <inertia ixx="0.002526666666667" ixy="0" ixz="0" iyy="0.002526666666667" iyz="0" izz="0.005"/>
-            </inertial>
-            <visual>
-                <geometry>
-                    <box size="0.05 0.01 0.01"/>
-                </geometry>
-            </visual>
-        </link>
-        <joint name="pitch_link_spring_${postfix}_joint" type="prismatic">
-            <origin xyz="0 0 0" rpy="0 0 0" />
-            <axis xyz="1 0 0" />
-            <parent link="pitch_link_${postfix}" />
-            <child link="spring_mount_${postfix}" />
-            <limit lower="0" upper="0.150" effort="1000" velocity="1000"/>
-        </joint>
-        <joint name="pitch_link_mount_${postfix}_joint" type="continuous">
-            <origin xyz="${x-0.012} 0 ${z-0.05367}" rpy="0 0 0" />
-            <axis xyz="0 1 0" />
-            <parent link="bottom_wheel_mount_${postfix}" />
-            <child link="pitch_link_${postfix}" />
-        </joint>
-    <!-- Spring mount -->
-        <link name="spring_mount_${postfix}">
-            <inertial>
-                <mass value="0.001" />
-                <inertia ixx="0.002526666666667" ixy="0" ixz="0" iyy="0.002526666666667" iyz="0" izz="0.005"/>
-            </inertial>
-            <visual>
-                <geometry>
-                    <box size="0.05 0.01 0.01"/>
-                </geometry>
-            </visual>
-        </link>
-        <joint name="spring_mount_${postfix}_joint" type="continuous">
-            <origin xyz="${x+0.17805} 0 ${z+0.01519}" rpy="0 0 0" />
-            <axis xyz="0 1 0"/>
-            <parent link="${parent}" />
-            <child link="spring_mount_${postfix}"/>
-        </joint>
     </xacro:macro>
 </robot>

Commit message: Suspension working

File: src/rr_robot_description/urdf/robot.urdf.xacro (robot description, xacro)
@@ -87,5 +87,5 @@
   <xacro:attach_tool_macro toolholder="th6" tool="$(arg th6_tool)" prefix="th6_"/>
   <xacro:attach_tool_macro toolholder="th7" tool="$(arg th7_tool)" prefix="th7_"/>
-  <!-- ******************************** Tranmissions ******************************** -->
+  <!-- ******************************** wheels ******************************** -->
   <xacro:include filename="$(find rr_robot_description)/urdf/wheel_assembly/bottom_wheel.xacro" />
   <xacro:bottom_wheels_macro parent="${robot_name}_chassis"

File: src/rr_robot_description/urdf/transmissions.xacro (robot description, xacro)
@@ -14,5 +14,5 @@
     <xacro:EffortJointMacro joint_name="rope_drive_le_joint"/>
     <xacro:EffortJointMacro joint_name="rope_drive_te_joint"/>
-    <xacro:EffortJointMacro joint_name="top_wheel_le_joint"/>
-    <xacro:EffortJointMacro joint_name="top_wheel_te_joint"/>
+    <xacro:EffortJointMacro joint_name="top_wheel_yaw_joint_te"/>
+    <xacro:EffortJointMacro joint_name="top_wheel_yaw_joint_le"/>
 </robot>

File: src/rr_robot_description/urdf/wheel_assembly/bottom_wheel.xacro (robot description, xacro)
@@ -33,4 +33,5 @@
                 <parent link="${parent}" />
                 <child link="bottom_wheel_mount_${postfix}"/>
+                <dynamics damping="1" />
             </joint>
         <!-- Wheel -->
@@ -61,4 +62,5 @@
                 <parent link="bottom_wheel_mount_${postfix}" />
                 <child link="bottom_wheel_${postfix}" />
+                <dynamics damping="1" />
             </joint>
         </xacro:macro>

File: src/rr_robot_description/urdf/wheel_assembly/top_wheel.xacro (robot description, xacro)
@@ -35,4 +35,5 @@
               <parent link="${parent}" />
               <child link="top_wheel_mount_${postfix}"/>
+              <dynamics damping="1" />
           </joint>
           <link name="yaw_link_${postfix}">
@@ -50,4 +51,5 @@
               <parent link="top_wheel_mount_${postfix}" />
               <child link="yaw_link_${postfix}" />
+              <dynamics damping="1" />
           </joint>
           <link name="top_wheel_${postfix}">
@@ -78,4 +80,5 @@
             <parent link="yaw_link_${postfix}" />
             <child link="top_wheel_${postfix}" />
+            <dynamics damping="1" />
           </joint>
         </xacro:macro>

Commit message: Suspension working

File: src/rr_robot_description/urdf/robot.urdf.xacro (robot description, xacro)
@@ -87,17 +87,19 @@
   <xacro:attach_tool_macro toolholder="th6" tool="$(arg th6_tool)" prefix="th6_"/>
   <xacro:attach_tool_macro toolholder="th7" tool="$(arg th7_tool)" prefix="th7_"/>
-  <!-- ******************************** Tranmissions ******************************** -->
+  <!-- ******************************** wheels ******************************** -->
   <xacro:include filename="$(find rr_robot_description)/urdf/wheel_assembly/bottom_wheel.xacro" />
   <xacro:bottom_wheels_macro parent="${robot_name}_chassis"
                             x= "-0.0251"
-                            wspan= "${2*0.1615}"
+                            wspan= "0.323"
                             z= "-0.11818"/>
   <xacro:include filename="$(find rr_robot_description)/urdf/wheel_assembly/top_wheel.xacro" />
   <xacro:top_wheels_macro parent="${robot_name}_chassis"
                             x= "1.13039"
-                            wspan= "${2*0.12962}"
+                            wspan= "0.342"
                             z= "-0.1344"/>
   <!-- ******************************** Tranmissions ******************************** -->
   <xacro:include filename="$(find rr_robot_description)/urdf/transmissions.xacro" />
+  <!--***************************** Rope for winch plugin *****************************-->
+  <xacro:include filename="$(find rr_robot_description)/urdf/rope.xacro" />
   <!-- *********************************** Gazebo *********************************** -->
   <xacro:include filename="$(find rr_robot_description)/urdf/robot.gazebo" />

File: src/rr_robot_description/urdf/rope.xacro (robot description, xacro)
@@ -2,4 +2,18 @@
 <robot xmlns:xacro="http://ros.org/wiki/xacro" name="rope_macro">
   <xacro:macro name="chassis_macro" params="parent_link">
+    <!-- Rope yaw -->
+    <link name="rope_yaw_link">
+        <inertial>
+          <mass value="0.01" />
+          <inertia ixx="0.01" ixy="0.0" ixz="0.0" iyy="0.01" iyz="0.0" izz="0.01" />
+        </inertial>
+    </link>
+    <joint name="rope_yaw_joint" type="revolute">
+      <axis xyz="0 0 1" />
+      <limit lower="-0.7853" upper="0.7853"/>
+      <parent link="${parent_link}"/>
+      <child link="rope_yaw_link"/>
+    </joint>
+    <!-- rope prismatic joint (springed joint)-->
     <link name="rope_link">
         <inertial>
@@ -8,21 +22,12 @@
           <inertia ixx="0.01" ixy="0.0" ixz="0.0" iyy="0.01" iyz="0.0" izz="0.01" />
         </inertial>
-        <visual>
-          <origin xyz="0 0 0" rpy="0 0 0" />
-          <geometry>
-            <empty></empty>
-          </geometry>
-        </visual>
-        <collision>
-          <origin xyz="0 0 0" rpy="0 0 0" />
-          <geometry>
-            <empty></empty>
-          </geometry>
-        </collision>
-      </link>
-      <joint name="${parent_link}_to_rope" type="floating">
-        <parent link="${parent_link}"/>
-        <child link="rope_link" />
-      </joint>
+    </link>
+    <joint name="${parent_link}_to_rope" type="prismatic">
+      <origin xyz="0 0 35" />
+      <axis xyz="1 0 0" />
+      <parent link="rope_yaw_link"/>
+      <child link="rope_link" />
+      <dynamics damping="1" />
+    </joint>
   </xacro:macro>
 </robot>
