Commit message: Fixed suspension

File: src/rr_robot_description/urdf/robot.urdf.xacro (robot description, xacro)
@@ -90,12 +90,12 @@
   <xacro:include filename="$(find rr_robot_description)/urdf/wheel_assembly/bot_wheel.xacro" />
   <xacro:bot_wheels_macro parent="${robot_name}_chassis"
-                            x= "-0.0251"
+                            x= "-0.0265"
                             wspan= "0.323"
                             z= "-0.11818"/>
   <xacro:include filename="$(find rr_robot_description)/urdf/wheel_assembly/top_wheel.xacro" />
   <xacro:top_wheels_macro parent="${robot_name}_chassis"
-                            x= "1.13039"
+                            x= "1.12508"
                             wspan= "0.342"
-                            z= "-0.1344"/>
+                            z= "-0.13492"/>
   <!-- ******************************** Tranmissions ******************************** -->
   <xacro:include filename="$(find rr_robot_description)/urdf/transmissions.xacro" />

File: src/rr_robot_description/urdf/wheel_assembly/bot_wheel.xacro (robot description, xacro)
@@ -1,4 +1,5 @@
 <?xml version="1.0"?>
-<!-- because closed loops are not allowed in URDF, the suspension is simplified to a torsional spring
+<!-- because closed loops are not allowed in URDF, the suspension is simplified to a torsional
+spring
     at the wheel mount revolute joint. This can approximate the more complicated suspension as long as
     the range of motion is small -->
@@ -15,34 +16,32 @@
                 <xacro:property name="y" value="${wspan/2}" />
             </xacro:unless>
-        <!-- Wheel mount -->
+            <!-- Wheel mount -->
             <link name="bot_wheel_mount_${postfix}">
                 <inertial>
                     <mass value="0.001" />
-                    <inertia ixx="0.002526666666667" ixy="0" ixz="0" iyy="0.002526666666667" iyz="0" izz="0.005"/>
+                    <inertia ixx="0.002526666666667" ixy="0" ixz="0" iyy="0.002526666666667" iyz="0"
+                        izz="0.005" />
                 </inertial>
-                <visual>
-                    <geometry>
-                        <box size="0.05 0.01 0.01"/>
-                    </geometry>
-                </visual>
             </link>
             <joint name="bot_pivot_joint_${postfix}" type="revolute">
                 <origin xyz="${x+0.06343} ${y} ${z+0.01419}" rpy="0 0 0" />
                 <axis xyz="0 1 0" />
-                <limit lower="${-range}" upper="${range}" effort="1000" velocity="1000"/>
+                <limit lower="${-range}" upper="${range}" effort="100000" velocity="1000" />
                 <parent link="${parent}" />
-                <child link="bot_wheel_mount_${postfix}"/>
-                <dynamics damping="30" friction="1" />
+                <child link="bot_wheel_mount_${postfix}" />
+                <dynamics damping="1" friction="1" />
             </joint>
-        <!-- Wheel -->
+            <!-- Wheel -->
             <link name="bot_wheel_${postfix}">
                 <inertial>
                     <mass value="1" />
-                    <inertia ixx="0.002526666666667" ixy="0" ixz="0" iyy="0.002526666666667" iyz="0" izz="0.005"/>
+                    <inertia ixx="0.002526666666667" ixy="0" ixz="0" iyy="0.002526666666667" iyz="0"
+                        izz="0.005" />
                 </inertial>
                 <visual>
                     <origin xyz="0 0 0" rpy="0 0 0" />
                     <geometry>
-                        <mesh filename="package://rr_robot_description/include/chassis/meshes/BottomWheels/visual.STL" />
+                        <mesh
+                            filename="package://rr_robot_description/include/chassis/meshes/BottomWheels/visual.STL" />
                     </geometry>
                     <material name="grey">
@@ -51,13 +50,14 @@
                 </visual>
                 <collision>
-                <origin xyz="0 0 0" rpy="0 0 0" />
-                <geometry>
-                    <mesh filename="package://rr_robot_description/include/chassis/meshes/BottomWheels/collision.STL" />
-                </geometry>
+                    <origin xyz="0 0 0" rpy="0 0 0" />
+                    <geometry>
+                        <mesh
+                            filename="package://rr_robot_description/include/chassis/meshes/BottomWheels/collision.STL" />
+                    </geometry>
                 </collision>
             </link>
             <joint name="bot_wheel_joint_${postfix}" type="continuous">
                 <origin xyz="-0.06343 0 -0.01419" rpy="0 0 1.5708" />
-                <axis xyz="1 0 0"/>
+                <axis xyz="1 0 0" />
                 <parent link="bot_wheel_mount_${postfix}" />
                 <child link="bot_wheel_${postfix}" />

File: src/rr_robot_description/urdf/wheel_assembly/top_wheel.xacro (robot description, xacro)
@@ -1,87 +1,88 @@
 <?xml version="1.0"?>
-<!-- because closed loops are not allowed in URDF, the suspension is simplified to a torsional spring
+<!-- because closed loops are not allowed in URDF, the suspension is simplified to a torsional
+spring
     at the wheel mount revolute joint. This can approximate the more complicated suspension as long as
     the range of motion is small -->
 <robot xmlns:xacro="http://ros.org/wiki/xacro" name="top_wheels">
-    <xacro:macro name="top_wheels_macro" params="parent x z wspan">
-    <xacro:property name="range" value="0.174533" />
-      <!-- Macro for making a single wheel-->
-      <xacro:macro name="make_wheel" params="te='true'">
-          <xacro:if value="${te}">
-            <xacro:property name="postfix" value="te" />
-            <xacro:property name="y" value="${-wspan/2}" />
-            <xacro:property name="yaw_arm" value="-0.041" />
-          </xacro:if>
-          <xacro:unless value="${te}">
-            <xacro:property name="postfix" value="le" />
-            <xacro:property name="y" value="${wspan/2}" />
-            <xacro:property name="yaw_arm" value="0.041" />
-          </xacro:unless>
-          <link name="top_wheel_mount_${postfix}">
-            <inertial>
-                <mass value="0.001" />
-                <inertia ixx="0.002526666666667" ixy="0" ixz="0" iyy="0.002526666666667" iyz="0" izz="0.005"/>
-            </inertial>
-            <visual>
-                <geometry>
-                    <box size="0.05 0.01 0.01"/>
-                </geometry>
-            </visual>
-          </link>
-          <joint name="top_pivot_joint_${postfix}" type="revolute">
-              <origin xyz="${x-0.10581} ${y-yaw_arm} ${z-0.01217}" rpy="0 0 0" />
-              <axis xyz="0 1 0" />
-              <limit lower="${-range}" upper="${range}" effort="10000000" velocity="100000"/>
-              <parent link="${parent}" />
-              <child link="top_wheel_mount_${postfix}"/>
-              <dynamics damping="30" friction="1"/>
-          </joint>
-          <link name="yaw_link_${postfix}">
-              <inertial>
-                  <mass value="1" />
-                  <origin xyz="0 0 0" rpy="0 0 0" />
-                  <inertia ixx="0.002526666666667" ixy="0" ixz="0" iyy="0.002526666666667" iyz="0" izz="0.005"/>
-              </inertial>
-          </link>
-          <joint name="top_wheel_yaw_joint_${postfix}" type="revolute">
-              <origin xyz="0.10581 0 0.01217" rpy="0. 0. 1.5708" />
-              <axis xyz="0 0 1" />
-              <limit lower="-0.20" upper="0.20" effort="1000000" velocity="1000" />
-              <parent link="top_wheel_mount_${postfix}" />
-              <child link="yaw_link_${postfix}" />
-              <dynamics damping="1"/>
-          </joint>
-          <link name="top_wheel_${postfix}">
-            <inertial>
-              <mass value="1" />
-              <origin xyz="0 0 0" rpy="0 0 0" />
-              <inertia ixx="0.002526666666667" ixy="0" ixz="0" iyy="0.002526666666667" iyz="0" izz="0.005"/>
-            </inertial>
-            <visual>
-              <origin xyz="0 0 0" rpy="0 0 0" />
-              <geometry>
-                <mesh filename="package://rr_robot_description/include/chassis/meshes/BottomWheels/visual.STL" />
-              </geometry>
-              <material name="grey">
-                <color rgba="0.4 0.4 0.4 1" />
-              </material>
-            </visual>
-            <collision>
-              <origin xyz="0 0 0" rpy="0 0 0" />
-              <geometry>
-                <mesh filename="package://rr_robot_description/include/chassis/meshes/TopWheels/collision.STL" />
-              </geometry>
-            </collision>
-          </link>
-          <joint name="top_wheel_joint_${postfix}" type="continuous">
-            <origin xyz="${yaw_arm} 0 0" />
-            <axis xyz="1 0 0" />
-            <parent link="yaw_link_${postfix}" />
-            <child link="top_wheel_${postfix}" />
-            <dynamics damping="1" />
-          </joint>
-        </xacro:macro>
-        <xacro:make_wheel te="true" />
-        <xacro:make_wheel te="false" />
+  <xacro:macro name="top_wheels_macro" params="parent x z wspan">
+    <!-- Macro for making a single wheel-->
+    <xacro:macro name="make_wheel" params="te='true'">
+      <xacro:property name="range" value="0.174533" />
+      <xacro:if value="${te}">
+        <xacro:property name="postfix" value="te" />
+        <xacro:property name="y" value="${-wspan/2}" />
+        <xacro:property name="yaw_arm" value="-0.041" />
+      </xacro:if>
+      <xacro:unless value="${te}">
+        <xacro:property name="postfix" value="le" />
+        <xacro:property name="y" value="${wspan/2}" />
+        <xacro:property name="yaw_arm" value="0.041" />
+      </xacro:unless>
+      <link name="top_wheel_mount_${postfix}">
+        <inertial>
+          <mass value="0.001" />
+          <inertia ixx="0.002526666666667" ixy="0" ixz="0" iyy="0.002526666666667" iyz="0"
+            izz="0.005" />
+        </inertial>
+      </link>
+      <joint name="top_pivot_joint_${postfix}" type="revolute">
+        <origin xyz="${x-0.10581} ${y-yaw_arm} ${z-0.01217}" rpy="0 0 0" />
+        <axis xyz="0 1 0" />
+        <limit lower="${-range}" upper="${range}" effort="10000000" velocity="100000" />
+        <parent link="${parent}" />
+        <child link="top_wheel_mount_${postfix}" />
+        <dynamics damping="1" friction="1" />
+      </joint>
+      <link name="yaw_link_${postfix}">
+        <inertial>
+          <mass value="1" />
+          <origin xyz="0 0 0" rpy="0 0 0" />
+          <inertia ixx="0.002526666666667" ixy="0" ixz="0" iyy="0.002526666666667" iyz="0"
+            izz="0.005" />
+        </inertial>
+      </link>
+      <joint name="top_wheel_yaw_joint_${postfix}" type="revolute">
+        <origin xyz="0.10581 0 0.01217" rpy="0. 0. 1.5708" />
+        <axis xyz="0 0 1" />
+        <limit lower="-0.20" upper="0.20" effort="1000000" velocity="1000" />
+        <parent link="top_wheel_mount_${postfix}" />
+        <child link="yaw_link_${postfix}" />
+        <dynamics damping="1" />
+      </joint>
+      <link name="top_wheel_${postfix}">
+        <inertial>
+          <mass value="1" />
+          <origin xyz="0 0 0" rpy="0 0 0" />
+          <inertia ixx="0.002526666666667" ixy="0" ixz="0" iyy="0.002526666666667" iyz="0"
+            izz="0.005" />
+        </inertial>
+        <visual>
+          <origin xyz="0 0 0" rpy="0 0 0" />
+          <geometry>
+            <mesh
+              filename="package://rr_robot_description/include/chassis/meshes/BottomWheels/visual.STL" />
+          </geometry>
+          <material name="grey">
+            <color rgba="0.4 0.4 0.4 1" />
+          </material>
+        </visual>
+        <collision>
+          <origin xyz="0 0 0" rpy="0 0 0" />
+          <geometry>
+            <mesh
+              filename="package://rr_robot_description/include/chassis/meshes/BottomWheels/collision.STL" />
+          </geometry>
+        </collision>
+      </link>
+      <joint name="top_wheel_joint_${postfix}" type="continuous">
+        <origin xyz="${yaw_arm} 0 0" />
+        <axis xyz="1 0 0" />
+        <parent link="yaw_link_${postfix}" />
+        <child link="top_wheel_${postfix}" />
+        <dynamics damping="1" />
+      </joint>
     </xacro:macro>
+    <xacro:make_wheel te="true" />
+    <xacro:make_wheel te="false" />
+  </xacro:macro>
 </robot>

Commit message: Updated suspension values

File: src/rr_robot_description/urdf/robot.urdf.xacro (robot description, xacro)
@@ -90,12 +90,12 @@
   <xacro:include filename="$(find rr_robot_description)/urdf/wheel_assembly/bot_wheel.xacro" />
   <xacro:bot_wheels_macro parent="${robot_name}_chassis"
-                            x= "-0.0265"
+                            x= "0.03762"
                             wspan= "0.323"
-                            z= "-0.11818"/>
+                            z= "-0.13465"/>
   <xacro:include filename="$(find rr_robot_description)/urdf/wheel_assembly/top_wheel.xacro" />
   <xacro:top_wheels_macro parent="${robot_name}_chassis"
-                            x= "1.12508"
+                            x= "1.02306"
                             wspan= "0.342"
-                            z= "-0.13492"/>
+                            z= "-0.147"/>
   <!-- ******************************** Tranmissions ******************************** -->
   <xacro:include filename="$(find rr_robot_description)/urdf/transmissions.xacro" />

File: src/rr_robot_description/urdf/wheel_assembly/bot_wheel.xacro (robot description, xacro)
@@ -25,7 +25,7 @@
             </link>
             <joint name="bot_pivot_joint_${postfix}" type="revolute">
-                <origin xyz="${x+0.06343} ${y} ${z+0.01419}" rpy="0 0 0" />
+                <origin xyz="${x} ${y} ${z}" rpy="0 0 0" />
                 <axis xyz="0 1 0" />
-                <limit lower="${-range}" upper="${range}" effort="100000" velocity="1000" />
+                <limit lower="0" upper="0.38659043" effort="100000" velocity="1000" />
                 <parent link="${parent}" />
                 <child link="bot_wheel_mount_${postfix}" />
@@ -52,5 +52,5 @@
                     <origin xyz="0 0 0" rpy="0 1.57079633 0" />
                     <geometry>
-                        <cylinder radius="0.05" length="0.02"/>
+                        <cylinder radius="0.055" length="0.03322"/>
                         <!-- <mesh
                             filename="package://rr_robot_description/include/chassis/meshes/BottomWheels/collision.STL" /> -->
@@ -59,5 +59,5 @@
             </link>
             <joint name="bot_wheel_joint_${postfix}" type="continuous">
-                <origin xyz="-0.06343 0 -0.01419" rpy="0 0 1.5708" />
+                <origin xyz="-0.06062042 0 -0.0234556" rpy="0 0 1.5708" />
                 <axis xyz="1 0 0" />
                 <parent link="bot_wheel_mount_${postfix}" />

File: src/rr_robot_description/urdf/wheel_assembly/top_wheel.xacro (robot description, xacro)
@@ -8,5 +8,4 @@
     <!-- Macro for making a single wheel-->
     <xacro:macro name="make_wheel" params="te='true'">
-      <xacro:property name="range" value="0.174533" />
       <xacro:if value="${te}">
         <xacro:property name="postfix" value="te" />
@@ -27,7 +26,7 @@
       </link>
       <joint name="top_pivot_joint_${postfix}" type="revolute">
-        <origin xyz="${x-0.10581} ${y-yaw_arm} ${z-0.01217}" rpy="0 0 0" />
+        <origin xyz="${x} ${y} ${z}" rpy="0 0 0" />
         <axis xyz="0 1 0" />
-        <limit lower="${-range}" upper="${range}" effort="10000" velocity="100" />
+        <limit lower="0" upper="0.20542525" effort="10000" velocity="100" />
         <parent link="${parent}" />
         <child link="top_wheel_mount_${postfix}" />
@@ -43,5 +42,5 @@
       </link>
       <joint name="top_wheel_yaw_joint_${postfix}" type="revolute">
-        <origin xyz="0.10581 0 0.01217" rpy="0. 0. 1.5708" />
+        <origin xyz="0.10141 0 0.066" rpy="0. 0. 1.5708" />
         <axis xyz="0 0 1" />
         <limit lower="-0.20" upper="0.20" effort="500" velocity="5" />

Commit message: Updated suspension values

File: src/rr_robot_description/urdf/robot.urdf.xacro (robot description, xacro)
@@ -90,12 +90,12 @@
   <xacro:include filename="$(find rr_robot_description)/urdf/wheel_assembly/bot_wheel.xacro" />
   <xacro:bot_wheels_macro parent="${robot_name}_chassis"
-                            x= "-0.0265"
+                            x= "0.03762"
                             wspan= "0.323"
-                            z= "-0.11818"/>
+                            z= "-0.13465"/>
   <xacro:include filename="$(find rr_robot_description)/urdf/wheel_assembly/top_wheel.xacro" />
   <xacro:top_wheels_macro parent="${robot_name}_chassis"
-                            x= "1.12508"
-                            wspan= "0.342"
-                            z= "-0.13492"/>
+                            x= "1.02306"
+                            wspan= "0.26"
+                            z= "-0.147"/>
   <!-- ******************************** Tranmissions ******************************** -->
   <xacro:include filename="$(find rr_robot_description)/urdf/transmissions.xacro" />

File: src/rr_robot_description/urdf/wheel_assembly/bot_wheel.xacro (robot description, xacro)
@@ -6,5 +6,4 @@
 <robot xmlns:xacro="http://ros.org/wiki/xacro" name="bot_wheel">
     <xacro:macro name="bot_wheels_macro" params="parent x z wspan">
-        <xacro:property name="range" value="0.174533" />
         <xacro:macro name="make_bot_wheel" params="te='true'">
             <xacro:if value="${te}">
@@ -25,7 +24,7 @@
             </link>
             <joint name="bot_pivot_joint_${postfix}" type="revolute">
-                <origin xyz="${x+0.06343} ${y} ${z+0.01419}" rpy="0 0 0" />
+                <origin xyz="${x} ${y} ${z}" rpy="0 0 0" />
                 <axis xyz="0 1 0" />
-                <limit lower="${-range}" upper="${range}" effort="100000" velocity="1000" />
+                <limit lower="0" upper="0.38659043" effort="100000" velocity="1000" />
                 <parent link="${parent}" />
                 <child link="bot_wheel_mount_${postfix}" />
@@ -52,5 +51,5 @@
                     <origin xyz="0 0 0" rpy="0 1.57079633 0" />
                     <geometry>
-                        <cylinder radius="0.05" length="0.02"/>
+                        <cylinder radius="0.055" length="0.03322"/>
                         <!-- <mesh
                             filename="package://rr_robot_description/include/chassis/meshes/BottomWheels/collision.STL" /> -->
@@ -59,5 +58,5 @@
             </link>
             <joint name="bot_wheel_joint_${postfix}" type="continuous">
-                <origin xyz="-0.06343 0 -0.01419" rpy="0 0 1.5708" />
+                <origin xyz="-0.06062042 0 -0.0234556" rpy="0 0 1.5708" />
                 <axis xyz="1 0 0" />
                 <parent link="bot_wheel_mount_${postfix}" />

File: src/rr_robot_description/urdf/wheel_assembly/top_wheel.xacro (robot description, xacro)
@@ -8,5 +8,4 @@
     <!-- Macro for making a single wheel-->
     <xacro:macro name="make_wheel" params="te='true'">
-      <xacro:property name="range" value="0.174533" />
       <xacro:if value="${te}">
         <xacro:property name="postfix" value="te" />
@@ -27,7 +26,7 @@
       </link>
       <joint name="top_pivot_joint_${postfix}" type="revolute">
-        <origin xyz="${x-0.10581} ${y-yaw_arm} ${z-0.01217}" rpy="0 0 0" />
+        <origin xyz="${x} ${y} ${z}" rpy="0 0 0" />
         <axis xyz="0 1 0" />
-        <limit lower="${-range}" upper="${range}" effort="10000" velocity="100" />
+        <limit lower="-0.20542525" upper="0" effort="10000" velocity="100" />
         <parent link="${parent}" />
         <child link="top_wheel_mount_${postfix}" />
@@ -43,7 +42,7 @@
       </link>
       <joint name="top_wheel_yaw_joint_${postfix}" type="revolute">
-        <origin xyz="0.10581 0 0.01217" rpy="0. 0. 1.5708" />
+        <origin xyz="0.10141 0 -0.066" rpy="0. 0. 1.5708" />
         <axis xyz="0 0 1" />
-        <limit lower="-0.20" upper="0.20" effort="500" velocity="5" />
+        <limit lower="0" upper="0.20" effort="500" velocity="5" />
         <parent link="top_wheel_mount_${postfix}" />
         <child link="yaw_link_${postfix}" />
@@ -70,5 +69,5 @@
           <origin xyz="0 0 0" rpy="0 1.57079633 0" />
           <geometry>
-            <cylinder radius="0.05" length="0.02"/>
+            <cylinder radius="0.055" length="0.02"/>
             <!-- <mesh
               filename="package://rr_robot_description/include/chassis/meshes/BottomWheels/collision.STL" /> -->

Commit message: small change

File: src/rr_robot_description/urdf/robot.urdf.xacro (robot description, xacro)
@@ -91,7 +91,5 @@
   <xacro:bot_wheels_macro parent="${robot_name}_chassis"
                             x= "0.03762"
-                            x= "0.03762"
                             wspan= "0.323"
-                            z= "-0.13465"/>
                             z= "-0.13465"/>
   <xacro:include filename="$(find rr_robot_description)/urdf/wheel_assembly/top_wheel.xacro" />

File: src/rr_robot_description/urdf/wheel_assembly/top_wheel.xacro (robot description, xacro)
@@ -43,5 +43,5 @@
       </link>
       <joint name="top_wheel_yaw_joint_${postfix}" type="revolute">
-        <origin xyz="0.10141 0 0.066" rpy="0. 0. 1.5708" />
+        <origin xyz="0.09941 0 0.02003" rpy="0. 0. 1.5708" />
         <axis xyz="0 0 1" />
         <limit lower="0" upper="0.20" effort="500" velocity="5" />
