Commit message: Collision of vacuum sheet neglected

File: src/rr_robot_description/include/chassis/urdf/chassis.xacro (robot description, xacro)
@@ -244,10 +244,11 @@
         </material>
       </visual>
-      <collision>
+      <!-- Collision of vacuum sheet is neglected -->
+      <!--<collision>
         <origin xyz="0 0 0" rpy="0 0 0" />
         <geometry>
           <mesh filename="package://rr_robot_description/include/chassis/meshes/VacuumSheet/collision.STL" />
         </geometry>
-      </collision>
+      </collision> -->
     </link>
     <joint name="vacuum_sheet_joint" type="fixed">

Commit message: winch plugin in progress

File: src/rr_robot_description/include/chassis/urdf/chassis.xacro (robot description, xacro)
@@ -244,10 +244,10 @@
         </material>
       </visual>
-      <collision>
+      <!-- <collision>
         <origin xyz="0 0 0" rpy="0 0 0" />
         <geometry>
           <mesh filename="package://rr_robot_description/include/chassis/meshes/VacuumSheet/collision.STL" />
         </geometry>
-      </collision>
+      </collision> -->
     </link>
     <joint name="vacuum_sheet_joint" type="fixed">

File: src/rr_robot_description/urdf/robot.urdf.xacro (robot description, xacro)
@@ -17,5 +17,5 @@
   <xacro:property name="arm_z_offset" value="0" />
   <!-- world base link -->
-  <link name="world">
+  <link name="dummy">
     <origin xyz="0 0 0" rpy="0 0 0"/>
   </link>
@@ -23,5 +23,5 @@
   <xacro:include filename="$(find rr_robot_description)/include/chassis/urdf/chassis.xacro" />
   <xacro:chassis_macro name="${robot_name}_chassis"
-                       parent_link="world"
+                       parent_link="dummy"
                        x_offset="-${arm_x_offset}"
                        y_offset="-${arm_y_offset}"

File: src/rr_robot_description/urdf/transmissions.xacro (robot description, xacro)
@@ -5,5 +5,5 @@
             <type>transmission_interface/SimpleTransmission</type>
             <joint name="${joint_name}">
-                <hardwareInterface>EffortJointInterface</hardwareInterface>
+                <hardwareInterface>hardware_interface/EffortJointInterface</hardwareInterface>
             </joint>
             <actuator name="${joint_name}_motor">

Commit message: "added bottom wheel xacro"

File: src/rr_robot_description/include/chassis/urdf/chassis.xacro (robot description, xacro)
@@ -227,4 +227,5 @@
       <child link="top_wheel_te" />
     </joint>
+    <!--  -->
     <!-- ********************* Vacuum Sheet ********************* -->
     <!-- TODO: add mass and inertia -->

File: src/rr_robot_description/urdf/robot.urdf.xacro (robot description, xacro)
@@ -88,4 +88,11 @@
   <xacro:attach_tool_macro toolholder="th7" tool="$(arg th7_tool)" prefix="th7_"/>
   <!-- ******************************** Tranmissions ******************************** -->
+  <xacro:include filename="$(find rr_robot_description)/urdf/wheel_assembly/bottom_wheel.xacro" />
+  <xacro:bottom_wheel_macro parent="${robot_name}_chassis"
+                            x= "-0.0251"
+                            y= "0.1615"
+                            z= "-0.11818"
+                            postfix="le" />
+  <!-- ******************************** Tranmissions ******************************** -->
   <xacro:include filename="$(find rr_robot_description)/urdf/transmissions.xacro" />
   <!-- *********************************** Gazebo *********************************** -->

File: src/rr_robot_description/urdf/suspension.xacro (robot description, xacro)
@@ -1,5 +1,5 @@
 <?xml version="1.0"?>
 <robot xmlns:xacro="http://ros.org/wiki/xacro" name="suspension">
-    <xacro:macro name="attach_tool_macro" params="parent">
+    <xacro:macro name="suspension_macro" params="parent">
         <link name="rope_drive_te">
             <inertial>

Commit message: Suspension working in rviz

File: src/rr_robot_description/include/chassis/urdf/chassis.xacro (robot description, xacro)
@@ -109,123 +109,4 @@
       <child link="rope_drive_te" />
     </joint>
-    <!-- ********************* Bottom Wheels ******************** -->
-    <!-- TODO: add mass and inertia -->
-    <link name="bot_wheel_le">
-      <inertial>
-        <mass value="1" />
-        <origin xyz="0 0 0" rpy="0 0 0" />
-        <inertia ixx="0.002526666666667" ixy="0" ixz="0" iyy="0.002526666666667" iyz="0" izz="0.005"/>
-      </inertial>
-      <visual>
-        <origin xyz="0 0 0" rpy="0 0 0" />
-        <geometry>
-          <mesh filename="package://rr_robot_description/include/chassis/meshes/BottomWheels/visual.STL" />
-        </geometry>
-        <material name="grey">
-          <color rgba="0.4 0.4 0.4 1" />
-        </material>
-      </visual>
-      <collision>
-        <origin xyz="0 0 0" rpy="0 0 0" />
-        <geometry>
-          <mesh filename="package://rr_robot_description/include/chassis/meshes/BottomWheels/collision.STL" />
-        </geometry>
-      </collision>
-    </link>
-    <joint name="bot_wheel_le_joint" type="fixed">
-      <origin xyz="-0.0251 0.1615 -0.11818" rpy="0. 0. 1.5708" />
-      <parent link="${name}" />
-      <child link="bot_wheel_le" />
-    </joint>
-    <link name="bot_wheel_te">
-      <inertial>
-        <mass value="1" />
-        <origin xyz="0 0 0" rpy="0 0 0" />
-        <inertia ixx="0.002526666666667" ixy="0" ixz="0" iyy="0.002526666666667" iyz="0" izz="0.005"/>
-      </inertial>
-      <visual>
-        <origin xyz="0 0 0" rpy="0 0 0" />
-        <geometry>
-          <mesh filename="package://rr_robot_description/include/chassis/meshes/BottomWheels/visual.STL" />
-        </geometry>
-        <material name="grey">
-          <color rgba="0.4 0.4 0.4 1" />
-        </material>
-      </visual>
-      <collision>
-        <origin xyz="0 0 0" rpy="0 0 0" />
-        <geometry>
-          <mesh filename="package://rr_robot_description/include/chassis/meshes/BottomWheels/collision.STL" />
-        </geometry>
-      </collision>
-    </link>
-    <joint name="bot_wheel_te_joint" type="fixed">
-      <origin xyz="-0.0251 -0.1615 -0.11818" rpy="0. 0. -1.5708" />
-      <parent link="${name}" />
-      <child link="bot_wheel_te" />
-    </joint>
-    <!-- ********************* Top Wheels *********************** -->
-    <!-- TODO: add mass and inertia -->
-    <link name="top_wheel_le">
-      <inertial>
-        <mass value="1" />
-        <origin xyz="0 0 0" rpy="0 0 0" />
-        <inertia ixx="0.002526666666667" ixy="0" ixz="0" iyy="0.002526666666667" iyz="0" izz="0.005"/>
-      </inertial>
-      <visual>
-        <origin xyz="0 0 0" rpy="0 0 0" />
-        <geometry>
-          <mesh filename="package://rr_robot_description/include/chassis/meshes/TopWheels/visual.STL" />
-        </geometry>
-        <material name="grey">
-          <color rgba="0.4 0.4 0.4 1" />
-        </material>
-      </visual>
-      <collision>
-        <origin xyz="0 0 0" rpy="0 0 0" />
-        <geometry>
-          <mesh filename="package://rr_robot_description/include/chassis/meshes/TopWheels/collision.STL" />
-        </geometry>
-      </collision>
-    </link>
-    <joint name="top_wheel_le_joint" type="revolute">
-      <origin xyz="1.13039 0.12962 -0.1344" rpy="0. 0. 1.5708" />
-      <axis rpy="0 0 0" xyz="0 0 1" />
-      <limit lower="-0.20" upper="0.20" effort="10000" velocity="1000" />
-      <joint_properties damping="1.0" friction="1.0" />
-      <parent link="${name}" />
-      <child link="top_wheel_le" />
-    </joint>
-    <link name="top_wheel_te">
-      <inertial>
-        <mass value="1" />
-        <origin xyz="0 0 0" rpy="0 0 0" />
-        <inertia ixx="0.002526666666667" ixy="0" ixz="0" iyy="0.002526666666667" iyz="0" izz="0.005"/>
-      </inertial>
-      <visual>
-        <origin xyz="0 0 0" rpy="0 0 0" />
-        <geometry>
-          <mesh filename="package://rr_robot_description/include/chassis/meshes/TopWheels/visual.STL" />
-        </geometry>
-        <material name="grey">
-          <color rgba="0.4 0.4 0.4 1" />
-        </material>
-      </visual>
-      <collision>
-        <origin xyz="0 0 0" rpy="0 0 0" />
-        <geometry>
-          <mesh filename="package://rr_robot_description/include/chassis/meshes/TopWheels/collision.STL" />
-        </geometry>
-      </collision>
-    </link>
-    <joint name="top_wheel_te_joint" type="revolute">
-      <origin xyz="1.13039 -0.12962 -0.1344" rpy="0. 0. -1.5708" />
-      <axis rpy="0 0 0" xyz="0 0 1" />
-      <limit lower="-0.20" upper="0.20" effort="10000" velocity="1000" />
-      <joint_properties damping="1.0" friction="1.0" />
-      <parent link="${name}" />
-      <child link="top_wheel_te" />
-    </joint>
-    <!--  -->
     <!-- ********************* Vacuum Sheet ********************* -->
     <!-- TODO: add mass and inertia -->

File: src/rr_robot_description/urdf/robot.urdf.xacro (robot description, xacro)
@@ -89,25 +89,13 @@
   <!-- ******************************** Tranmissions ******************************** -->
   <xacro:include filename="$(find rr_robot_description)/urdf/wheel_assembly/bottom_wheel.xacro" />
-  <xacro:bottom_wheel_macro parent="${robot_name}_chassis"
+  <xacro:bottom_wheels_macro parent="${robot_name}_chassis"
                             x= "-0.0251"
-                            y= "0.1615"
-                            z= "-0.11818"
-                            postfix="le" />
-  <xacro:bottom_wheel_macro parent="${robot_name}_chassis"
-                            x= "-0.0251"
-                            y= "-0.1615"
-                            z= "-0.11818"
-                            postfix="te" />
+                            wspan= "${2*0.1615}"
+                            z= "-0.11818"/>
   <xacro:include filename="$(find rr_robot_description)/urdf/wheel_assembly/top_wheel.xacro" />
-  <xacro:top_wheel_macro parent="${robot_name}_chassis"
+  <xacro:top_wheels_macro parent="${robot_name}_chassis"
                             x= "1.13039"
-                            y= "0.12962"
-                            z= "-0.1344"
-                            postfix="le" />
-  <xacro:top_wheel_macro parent="${robot_name}_chassis"
-                            x= "1.13039"
-                            y= "-0.12962"
-                            z= "-0.1344"
-                            postfix="te" />
+                            wspan= "${2*0.12962}"
+                            z= "-0.1344"/>
   <!-- ******************************** Tranmissions ******************************** -->
   <xacro:include filename="$(find rr_robot_description)/urdf/transmissions.xacro" />

File: src/rr_robot_description/urdf/wheel_assembly/bottom_wheel.xacro (robot description, xacro)
@@ -5,52 +5,64 @@
 <robot xmlns:xacro="http://ros.org/wiki/xacro" name="bot_wheel">
     <xacro:property name="range" value="0.174533" />
-    <xacro:macro name="bottom_wheel_macro" params="parent x y z postfix">
-    <!-- Wheel mount -->
-        <link name="bottom_wheel_mount_${postfix}">
-            <inertial>
-                <mass value="0.001" />
-                <inertia ixx="0.002526666666667" ixy="0" ixz="0" iyy="0.002526666666667" iyz="0" izz="0.005"/>
-            </inertial>
-            <visual>
+    <xacro:macro name="bottom_wheels_macro" params="parent x z wspan">
+        <xacro:macro name="make_bottom_wheel" params="te='true'">
+            <xacro:if value="${te}">
+                <xacro:property name="postfix" value="te" />
+                <xacro:property name="y" value="${-wspan/2}" />
+            </xacro:if>
+            <xacro:unless value="${te}">
+                <xacro:property name="postfix" value="le" />
+                <xacro:property name="y" value="${wspan/2}" />
+            </xacro:unless>
+        <!-- Wheel mount -->
+            <link name="bottom_wheel_mount_${postfix}">
+                <inertial>
+                    <mass value="0.001" />
+                    <inertia ixx="0.002526666666667" ixy="0" ixz="0" iyy="0.002526666666667" iyz="0" izz="0.005"/>
+                </inertial>
+                <visual>
+                    <geometry>
+                        <box size="0.05 0.01 0.01"/>
+                    </geometry>
+                </visual>
+            </link>
+            <joint name="bottom_pivot_joint_${postfix}" type="revolute">
+                <origin xyz="${x+0.06343} ${y} ${z+0.01419}" rpy="0 0 0" />
+                <axis xyz="0 1 0" />
+                <limit lower="${-range}" upper="${range}" effort="1000" velocity="1000"/>
+                <parent link="${parent}" />
+                <child link="bottom_wheel_mount_${postfix}"/>
+            </joint>
+        <!-- Wheel -->
+            <link name="bottom_wheel_${postfix}">
+                <inertial>
+                    <mass value="1" />
+                    <inertia ixx="0.002526666666667" ixy="0" ixz="0" iyy="0.002526666666667" iyz="0" izz="0.005"/>
+                </inertial>
+                <visual>
+                    <origin xyz="0 0 0" rpy="0 0 0" />
+                    <geometry>
+                        <mesh filename="package://rr_robot_description/include/chassis/meshes/BottomWheels/visual.STL" />
+                    </geometry>
+                    <material name="grey">
+                        <color rgba="0.4 0.4 0.4 1" />
+                    </material>
+                </visual>
+                <collision>
+                <origin xyz="0 0 0" rpy="0 0 0" />
                 <geometry>
-                    <box size="0.05 0.01 0.01"/>
+                    <mesh filename="package://rr_robot_description/include/chassis/meshes/BottomWheels/collision.STL" />
                 </geometry>
-            </visual>
-        </link>
-        <joint name="bottom_pivot_joint_${postfix}" type="revolute">
-            <origin xyz="${x+0.06343} ${y} ${z+0.01419}" rpy="0 0 0" />
-            <axis xyz="0 1 0" />
-            <limit lower="${-range}" upper="${range}" effort="1000" velocity="1000"/>
-            <parent link="${parent}" />
-            <child link="bottom_wheel_mount_${postfix}"/>
-        </joint>
-    <!-- Wheel -->
-        <link name="bottom_wheel_${postfix}">
-            <inertial>
-                <mass value="1" />
-                <inertia ixx="0.002526666666667" ixy="0" ixz="0" iyy="0.002526666666667" iyz="0" izz="0.005"/>
-            </inertial>
-            <visual>
-              <origin xyz="0 0 0" rpy="0 0 0" />
-              <geometry>
-                <mesh filename="package://rr_robot_description/include/chassis/meshes/BottomWheels/visual.STL" />
-              </geometry>
-              <material name="grey">
-                <color rgba="0.4 0.4 0.4 1" />
-              </material>
-            </visual>
-            <collision>
-              <origin xyz="0 0 0" rpy="0 0 0" />
-              <geometry>
-                <mesh filename="package://rr_robot_description/include/chassis/meshes/BottomWheels/collision.STL" />
-              </geometry>
-            </collision>
-        </link>
-        <joint name="bottom_wheel_joint_${postfix}" type="continuous">
-            <origin xyz="-0.06343 0 -0.01419" rpy="0 0 0" />
-            <axis xyz="0 1 0"/>
-            <parent link="bottom_wheel_mount_${postfix}" />
-            <child link="bottom_wheel_${postfix}" />
-        </joint>
+                </collision>
+            </link>
+            <joint name="bottom_wheel_joint_${postfix}" type="continuous">
+                <origin xyz="-0.06343 0 -0.01419" rpy="0 0 1.5708" />
+                <axis xyz="1 0 0"/>
+                <parent link="bottom_wheel_mount_${postfix}" />
+                <child link="bottom_wheel_${postfix}" />
+            </joint>
+        </xacro:macro>
+        <xacro:make_bottom_wheel te="true" />
+        <xacro:make_bottom_wheel te="false" />
     </xacro:macro>
 </robot>

File: src/rr_robot_description/urdf/wheel_assembly/top_wheel.xacro (robot description, xacro)
@@ -3,8 +3,20 @@
     at the wheel mount revolute joint. This can approximate the more complicated suspension as long as
     the range of motion is small -->
-<robot xmlns:xacro="http://ros.org/wiki/xacro" name="top_wheel">
+<robot xmlns:xacro="http://ros.org/wiki/xacro" name="top_wheels">
     <xacro:property name="range" value="0.174533" />
-    <xacro:macro name="top_wheel_macro" params="parent x y z postfix">
-        <link name="top_wheel_mount_${postfix}">
+    <xacro:macro name="top_wheels_macro" params="parent x z wspan">
+      <!-- Macro for making a single wheel-->
+      <xacro:macro name="make_wheel" params="te='true'">
+          <xacro:if value="${te}">
+            <xacro:property name="postfix" value="te" />
+            <xacro:property name="y" value="${-wspan/2}" />
+            <xacro:property name="yaw_arm" value="-0.041" />
+          </xacro:if>
+          <xacro:unless value="${te}">
+            <xacro:property name="postfix" value="le" />
+            <xacro:property name="y" value="${wspan/2}" />
+            <xacro:property name="yaw_arm" value="0.041" />
+          </xacro:unless>
+          <link name="top_wheel_mount_${postfix}">
             <inertial>
                 <mass value="0.001" />
@@ -16,28 +28,28 @@
                 </geometry>
             </visual>
-        </link>
-        <joint name="top_pivot_joint_${postfix}" type="revolute">
-            <origin xyz="${x-0.10581} ${y-41} ${z-0.01217}" rpy="0 0 0" />
-            <axis xyz="0 1 0" />
-            <limit lower="${-range}" upper="${range}" effort="1000" velocity="1000"/>
-            <parent link="${parent}" />
-            <child link="bottom_wheel_mount_${postfix}"/>
-        </joint>
-        <link name="yaw_link_${postfix}">
-            <inertial>
-                <mass value="1" />
-                <origin xyz="0 0 0" rpy="0 0 0" />
-                <inertia ixx="0.002526666666667" ixy="0" ixz="0" iyy="0.002526666666667" iyz="0" izz="0.005"/>
-            </inertial>
-        </link>
-        <joint name="top_wheel_yaw_joint_${postfix}" type="revolute">
-            <origin xyz="0.10581 0 0.01217" rpy="0. 0. 1.5708" />
-            <axis xyz="0 0 1" />
-            <limit lower="-0.20" upper="0.20" effort="10000" velocity="1000" />
-            <joint_properties damping="1.0" friction="1.0" />
-            <parent link="top_wheel_mount_${postfix}" />
-            <child link="yaw_link_${postfix}" />
-        </joint>
-        <link name="top_wheel_${postfix}">
+          </link>
+          <joint name="top_pivot_joint_${postfix}" type="revolute">
+              <origin xyz="${x-0.10581} ${y-yaw_arm} ${z-0.01217}" rpy="0 0 0" />
+              <axis xyz="0 1 0" />
+              <limit lower="${-range}" upper="${range}" effort="1000" velocity="1000"/>
+              <parent link="${parent}" />
+              <child link="top_wheel_mount_${postfix}"/>
+          </joint>
+          <link name="yaw_link_${postfix}">
+              <inertial>
+                  <mass value="1" />
+                  <origin xyz="0 0 0" rpy="0 0 0" />
+                  <inertia ixx="0.002526666666667" ixy="0" ixz="0" iyy="0.002526666666667" iyz="0" izz="0.005"/>
+              </inertial>
+          </link>
+          <joint name="top_wheel_yaw_joint_${postfix}" type="revolute">
+              <origin xyz="0.10581 0 0.01217" rpy="0. 0. 1.5708" />
+              <axis xyz="0 0 1" />
+              <limit lower="-0.20" upper="0.20" effort="10000" velocity="1000" />
+              <joint_properties damping="1.0" friction="1.0" />
+              <parent link="top_wheel_mount_${postfix}" />
+              <child link="yaw_link_${postfix}" />
+          </joint>
+          <link name="top_wheel_${postfix}">
             <inertial>
               <mass value="1" />
@@ -48,5 +60,5 @@
               <origin xyz="0 0 0" rpy="0 0 0" />
               <geometry>
-                <mesh filename="package://rr_robot_description/include/chassis/meshes/TopWheels/visual.STL" />
+                <mesh filename="package://rr_robot_description/include/chassis/meshes/BottomWheels/visual.STL" />
               </geometry>
               <material name="grey">
@@ -61,10 +73,13 @@
             </collision>
           </link>
-          <joint name="top_wheel_le_joint" type="continuous">
-            <origin xyz="0 41 0" />
-            <axis rpy="0 0 0" xyz="0 1 0" />
+          <joint name="top_wheel_joint_${postfix}" type="continuous">
+            <origin xyz="${yaw_arm} 0 0" />
+            <axis xyz="1 0 0" />
             <parent link="yaw_link_${postfix}" />
             <child link="top_wheel_${postfix}" />
           </joint>
+        </xacro:macro>
+        <xacro:make_wheel te="true" />
+        <xacro:make_wheel te="false" />
     </xacro:macro>
 </robot>
