Commit message: "rope plugin working"

File: src/rr_robot_description/include/chassis/urdf/chassis.xacro (robot description, xacro)
@@ -62,5 +62,5 @@
       </collision>
     </link>
-    <joint name="rope_drive_le_joint" type="continuous">
+    <joint name="rope_drive_le_joint" type="fixed">
       <origin xyz="0.92999 0.24067 -0.0269" rpy="-0.09857 0.09857 -1.64405" />
       <axis rpy="0 0 0" xyz="1 0 0" />
@@ -101,5 +101,5 @@
       </collision>
     </link>
-    <joint name="rope_drive_te_joint" type="continuous">
+    <joint name="rope_drive_te_joint" type="fixed">
       <origin xyz="0.92999 -0.24067 -0.0269" rpy="0.09857 0.09857 1.64405" />
       <axis rpy="0 0 0" xyz="1 0 0" />

File: src/rr_robot_description/urdf/robot.urdf.xacro (robot description, xacro)
@@ -88,6 +88,6 @@
   <xacro:attach_tool_macro toolholder="th7" tool="$(arg th7_tool)" prefix="th7_"/>
   <!-- ******************************** wheels ******************************** -->
-  <xacro:include filename="$(find rr_robot_description)/urdf/wheel_assembly/bottom_wheel.xacro" />
-  <xacro:bottom_wheels_macro parent="${robot_name}_chassis"
+  <xacro:include filename="$(find rr_robot_description)/urdf/wheel_assembly/bot_wheel.xacro" />
+  <xacro:bot_wheels_macro parent="${robot_name}_chassis"
                             x= "-0.0251"
                             wspan= "0.323"
@@ -102,4 +102,6 @@
   <!--***************************** Rope for winch plugin *****************************-->
   <xacro:include filename="$(find rr_robot_description)/urdf/rope.xacro" />
+  <xacro:rope_macro winch_name_no_postfix="rope_drive"
+                    rope_l="50"/>
   <!-- *********************************** Gazebo *********************************** -->
   <xacro:include filename="$(find rr_robot_description)/urdf/robot.gazebo" />

File: src/rr_robot_description/urdf/rope.xacro (robot description, xacro)
@@ -1,33 +1,67 @@
 <?xml version="1.0"?>
 <robot xmlns:xacro="http://ros.org/wiki/xacro" name="rope_macro">
-  <xacro:macro name="chassis_macro" params="parent_link">
-    <!-- Rope yaw -->
-    <link name="rope_yaw_link">
-        <inertial>
-          <mass value="0.01" />
-          <inertia ixx="0.01" ixy="0.0" ixz="0.0" iyy="0.01" iyz="0.0" izz="0.01" />
-        </inertial>
-    </link>
-    <joint name="rope_yaw_joint" type="revolute">
-      <axis xyz="0 0 1" />
-      <limit lower="-0.7853" upper="0.7853"/>
-      <parent link="${parent_link}"/>
-      <child link="rope_yaw_link"/>
-    </joint>
-    <!-- rope prismatic joint (springed joint)-->
-    <link name="rope_link">
-        <inertial>
-          <origin xyz="0.45171 -1.9114E-06 -0.0060107" rpy="0 0 0" />
-          <mass value="0.01" />
-          <inertia ixx="0.01" ixy="0.0" ixz="0.0" iyy="0.01" iyz="0.0" izz="0.01" />
-        </inertial>
-    </link>
-    <joint name="${parent_link}_to_rope" type="prismatic">
-      <origin xyz="0 0 35" />
-      <axis xyz="1 0 0" />
-      <parent link="rope_yaw_link"/>
-      <child link="rope_link" />
-      <dynamics damping="1" />
-    </joint>
+  <xacro:macro name="rope_macro" params="winch_name_no_postfix rope_l">
+    <xacro:macro name="make_rope" params="te='true'">
+      <xacro:if value="${te}" >
+        <xacro:property name="yaw" value="3.14159" />
+        <xacro:property name="postfix" value="te"/>
+      </xacro:if>
+      <xacro:unless value="${te}" >
+        <xacro:property name="yaw" value="0" />
+        <xacro:property name="postfix" value="le"/>
+      </xacro:unless>
+        <!-- Rope yaw -->
+        <link name="rope_yaw_link_${postfix}">
+          <inertial>
+            <mass value="0.01" />
+            <inertia ixx="0.01" ixy="0.0" ixz="0.0" iyy="0.01" iyz="0.0" izz="0.01" />
+          </inertial>
+      </link>
+      <joint name="rope_yaw_${postfix}_joint" type="revolute">
+        <axis xyz="0 0 1" />
+        <limit lower="-0.5235" upper="0.5235" effort="100000" velocity="1000000"/>
+        <parent link="${winch_name_no_postfix}_${postfix}"/>
+        <child link="rope_yaw_link_${postfix}"/>
+        <dynamics damping="0.5" />
+      </joint>
+      <!-- Rope pitch -->
+        <link name="rope_pitch_link_${postfix}">
+            <inertial>
+              <mass value="0.01" />
+              <inertia ixx="0.01" ixy="0.0" ixz="0.0" iyy="0.01" iyz="0.0" izz="0.01" />
+            </inertial>
+        </link>
+        <joint name="rope_pitch_${postfix}_joint" type="revolute">
+          <axis xyz="1 0 0" />
+          <limit lower="-0.5235" upper="0.5235" effort="100000" velocity="1000000"/>
+          <parent link="rope_yaw_link_${postfix}"/>
+          <child link="rope_pitch_link_${postfix}"/>
+          <dynamics damping="0.5" />
+        </joint>
+      <!-- rope prismatic joint (springed joint)-->
+      <link name="rope_link_${postfix}">
+          <inertial>
+            <origin rpy="1.57 0 0" />
+            <mass value="0.01" />
+            <inertia ixx="0.01" ixy="0.0" ixz="0.0" iyy="0.01" iyz="0.0" izz="0.01" />
+          </inertial>
+          <visual>
+            <origin rpy="1.57 0 0" />
+            <geometry>
+              <cylinder radius="0.01" length="0.5" />
+            </geometry>
+          </visual>
+      </link>
+      <joint name="rope_springed_joint_${postfix}" type="prismatic">
+        <origin xyz="0 0 0.035" rpy="0 0 ${yaw}" />
+        <axis xyz="0 1 0" />
+        <limit lower="0" upper="${rope_l}" effort="100000" velocity="1000000"/>
+        <parent link="rope_pitch_link_${postfix}"/>
+        <child link="rope_link_${postfix}" />
+        <dynamics damping="0.5" />
+      </joint>
+    </xacro:macro>
+    <xacro:make_rope te="true" />
+    <xacro:make_rope te="false" />
   </xacro:macro>
 </robot>

File: src/rr_robot_description/urdf/transmissions.xacro (robot description, xacro)
@@ -12,6 +12,6 @@
         </transmission>
     </xacro:macro>
-    <xacro:EffortJointMacro joint_name="rope_drive_le_joint"/>
-    <xacro:EffortJointMacro joint_name="rope_drive_te_joint"/>
+    <!-- <xacro:EffortJointMacro joint_name="rope_drive_le_joint"/>
+    <xacro:EffortJointMacro joint_name="rope_drive_te_joint"/> -->
     <xacro:EffortJointMacro joint_name="top_wheel_yaw_joint_te"/>
     <xacro:EffortJointMacro joint_name="top_wheel_yaw_joint_le"/>

File: src/rr_robot_description/urdf/wheel_assembly/bot_wheel.xacro (robot description, xacro)
@@ -5,6 +5,6 @@
 <robot xmlns:xacro="http://ros.org/wiki/xacro" name="bot_wheel">
     <xacro:property name="range" value="0.174533" />
-    <xacro:macro name="bottom_wheels_macro" params="parent x z wspan">
-        <xacro:macro name="make_bottom_wheel" params="te='true'">
+    <xacro:macro name="bot_wheels_macro" params="parent x z wspan">
+        <xacro:macro name="make_bot_wheel" params="te='true'">
             <xacro:if value="${te}">
                 <xacro:property name="postfix" value="te" />
@@ -16,5 +16,5 @@
             </xacro:unless>
         <!-- Wheel mount -->
-            <link name="bottom_wheel_mount_${postfix}">
+            <link name="bot_wheel_mount_${postfix}">
                 <inertial>
                     <mass value="0.001" />
@@ -27,14 +27,14 @@
                 </visual>
             </link>
-            <joint name="bottom_pivot_joint_${postfix}" type="revolute">
+            <joint name="bot_pivot_joint_${postfix}" type="revolute">
                 <origin xyz="${x+0.06343} ${y} ${z+0.01419}" rpy="0 0 0" />
                 <axis xyz="0 1 0" />
                 <limit lower="${-range}" upper="${range}" effort="1000" velocity="1000"/>
                 <parent link="${parent}" />
-                <child link="bottom_wheel_mount_${postfix}"/>
+                <child link="bot_wheel_mount_${postfix}"/>
                 <dynamics damping="1" />
             </joint>
         <!-- Wheel -->
-            <link name="bottom_wheel_${postfix}">
+            <link name="bot_wheel_${postfix}">
                 <inertial>
                     <mass value="1" />
@@ -44,5 +44,5 @@
                     <origin xyz="0 0 0" rpy="0 0 0" />
                     <geometry>
-                        <mesh filename="package://rr_robot_description/include/chassis/meshes/BottomWheels/visual.STL" />
+                        <mesh filename="package://rr_robot_description/include/chassis/meshes/botWheels/visual.STL" />
                     </geometry>
                     <material name="grey">
@@ -53,18 +53,18 @@
                 <origin xyz="0 0 0" rpy="0 0 0" />
                 <geometry>
-                    <mesh filename="package://rr_robot_description/include/chassis/meshes/BottomWheels/collision.STL" />
+                    <mesh filename="package://rr_robot_description/include/chassis/meshes/botWheels/collision.STL" />
                 </geometry>
                 </collision>
             </link>
-            <joint name="bottom_wheel_joint_${postfix}" type="continuous">
+            <joint name="bot_wheel_joint_${postfix}" type="continuous">
                 <origin xyz="-0.06343 0 -0.01419" rpy="0 0 1.5708" />
                 <axis xyz="1 0 0"/>
-                <parent link="bottom_wheel_mount_${postfix}" />
-                <child link="bottom_wheel_${postfix}" />
+                <parent link="bot_wheel_mount_${postfix}" />
+                <child link="bot_wheel_${postfix}" />
                 <dynamics damping="1" />
             </joint>
         </xacro:macro>
-        <xacro:make_bottom_wheel te="true" />
-        <xacro:make_bottom_wheel te="false" />
+        <xacro:make_bot_wheel te="true" />
+        <xacro:make_bot_wheel te="false" />
     </xacro:macro>
 </robot>

Commit message: Manual merge w new pkg. Added mass and inertias

File: src/rr_robot_description/include/chassis/urdf/chassis.xacro (robot description, xacro)
@@ -29,11 +29,39 @@
       <origin xyz="${x_offset} ${y_offset} ${z_offset}" rpy="0 0 0" />
     </joint>
+    <!-- ******************** IMU ******************************* -->
+    <!-- imu link -->
+    <link name="imu_link">
+      <inertial>
+        <mass value="0.1" />
+        <origin xyz="0 0 0" rpy="0 0 0" />
+        <inertia ixx="0.0001" ixy="0" ixz="0" iyy="0.0001" iyz="0" izz="0.0001"/>
+      </inertial>
+      <visual>
+        <origin xyz="0 0 0" rpy="0 0 0" />
+        <geometry>
+          <box size="0.03 0.03 0.03" />
+        </geometry>
+        <material name="grey">
+          <color rgba="0.4 0.4 0.4 1" />
+        </material>
+      </visual>
+      <collision>
+        <origin xyz="0 0 0" rpy="0 0 0" />
+        <geometry>
+          <box size="0.03 0.03 0.03" />
+        </geometry>
+      </collision>
+    </link>
+    <joint name="imu_joint" type="fixed">
+      <origin xyz="0.9 -0.035 0.093" rpy="0 ${pi} 0"/>
+      <parent link="${name}"/>
+      <child link="imu_link"/>
+    </joint>
     <!-- ********************* Rope Drives ********************** -->
-    <!-- TODO: add mass and inertia -->
     <link name="rope_drive_le">
       <inertial>
-        <mass value="1" />
-        <origin xyz="0 0 0" rpy="0 0 0" />
-        <inertia ixx="0.002526666666667" ixy="0" ixz="0" iyy="0.002526666666667" iyz="0" izz="0.005"/>
+        <mass value="2.206" />
+        <origin xyz="0.01032 0 0" rpy="0 0 0" />
+        <inertia ixx="0.00699387" ixy="0" ixz="0" iyy="0.0044146" iyz="0" izz="0.0044146"/>
       </inertial>
       <visual>
@@ -44,13 +72,4 @@
         <material name="grey">
           <color rgba="0.4 0.4 0.4 1" />
-        </material>
-      </visual>
-      <visual>
-        <origin rpy="${pi/2} 0 0" xyz="0.035 0 0" />
-        <geometry>
-          <box size="0.005 0.10 0.005" />
-        </geometry>
-        <material name="Grey">
-          <color rgba="0.6 0.6 0.6 1" />
         </material>
       </visual>
@@ -72,7 +91,7 @@
     <link name="rope_drive_te">
       <inertial>
-        <mass value="1" />
+        <mass value="2.206" />
         <origin xyz="0 0 0" rpy="0 0 0" />
-        <inertia ixx="0.002526666666667" ixy="0" ixz="0" iyy="0.002526666666667" iyz="0" izz="0.005"/>
+        <inertia ixx="0.00699387" ixy="0" ixz="0" iyy="0.0044146" iyz="0" izz="0.0044146"/>
       </inertial>
       <visual>
@@ -83,13 +102,4 @@
         <material name="grey">
           <color rgba="0.4 0.4 0.4 1" />
-        </material>
-      </visual>
-      <visual>
-        <origin rpy="${pi/2} 0 0" xyz="0.035 0 0" />
-        <geometry>
-          <box size="0.005 0.10 0.005" />
-        </geometry>
-        <material name="Grey">
-          <color rgba="0.6 0.6 0.6 1" />
         </material>
       </visual>
@@ -110,10 +120,9 @@
     </joint>
     <!-- ********************* Vacuum Sheet ********************* -->
-    <!-- TODO: add mass and inertia -->
     <link name="vacuum_sheet">
       <inertial>
-        <mass value="1" />
+        <mass value="0.6" />
         <origin xyz="0 0 0" rpy="0 0 0" />
-        <inertia ixx="0.002526666666667" ixy="0" ixz="0" iyy="0.002526666666667" iyz="0" izz="0.005"/>
+        <inertia ixx="0.0025275579" ixy="0" ixz="0" iyy="0.00001388" iyz="0" izz="0.04124286"/>
       </inertial>
       <visual>
@@ -162,238 +171,13 @@
     </joint>
     <!-- ********************* Tool holders ********************* -->
-    <link name="th0" >
-      <inertial>
-        <mass value="0.1911" />
-        <origin xyz="0 0 0" rpy="0 0 0" />
-        <inertia ixx="0.01880039566" ixy="-0.00288516792" ixz="0.00164510501" iyy="0.00519681040" iyz="-0.00798447007" izz="0.01485438661"/>
-      </inertial>
-      <visual>
-        <origin xyz="0 0 0" rpy="0 0 0" />
-        <geometry>
-          <mesh filename="package://rr_robot_description/include/chassis/meshes/ToolHolder/visual.STL" />
-        </geometry>
-        <material name="black">
-          <color rgba="0.2 0.2 0.2 1" />
-        </material>
-      </visual>
-      <collision>
-        <origin xyz="0 0 0" rpy="0 0 0" />
-        <geometry>
-          <mesh filename="package://rr_robot_description/include/chassis/meshes/ToolHolder/collision.STL" />
-        </geometry>
-      </collision>
-    </link>
-    <joint name="th0_joint" type="fixed">
-      <origin
-        xyz="0.95394 0.0875 0.12783"
-        rpy="-1.0611E-15 7.6478E-16 1.5708" />
-      <parent link="${name}" />
-      <child link="th0" />
-    </joint>
-    <link name="th1" >
-      <inertial>
-        <mass value="0.1911" />
-        <origin xyz="0 0 0" rpy="0 0 0" />
-        <inertia ixx="0.01880039566" ixy="-0.00288516792" ixz="0.00164510501" iyy="0.00519681040" iyz="-0.00798447007" izz="0.01485438661"/>
-      </inertial>
-      <visual>
-        <origin xyz="0 0 0" rpy="0 0 0" />
-        <geometry>
-          <mesh filename="package://rr_robot_description/include/chassis/meshes/ToolHolder/visual.STL" />
-        </geometry>
-        <material name="black">
-          <color rgba="0.2 0.2 0.2 1" />
-        </material>
-      </visual>
-      <collision>
-        <origin xyz="0 0 0" rpy="0 0 0" />
-        <geometry>
-          <mesh filename="package://rr_robot_description/include/chassis/meshes/ToolHolder/collision.STL" />
-        </geometry>
-      </collision>
-    </link>
-    <joint name="th1_joint" type="fixed">
-      <origin
-        xyz="0.95394 -0.0875 0.12783"
-        rpy="-1.0611E-15 7.6478E-16 1.5708" />
-      <parent link="${name}" />
-      <child link="th1" />
-    </joint>
-    <link name="th2" >
-      <inertial>
-        <mass value="0.1911" />
-        <origin xyz="0 0 0" rpy="0 0 0" />
-        <inertia ixx="0.01880039566" ixy="-0.00288516792" ixz="0.00164510501" iyy="0.00519681040" iyz="-0.00798447007" izz="0.01485438661"/>
-      </inertial>
-      <visual>
-        <origin xyz="0 0 0" rpy="0 0 0" />
-        <geometry>
-          <mesh filename="package://rr_robot_description/include/chassis/meshes/ToolHolder/visual.STL" />
-        </geometry>
-        <material name="black">
-          <color rgba="0.2 0.2 0.2 1" />
-        </material>
-      </visual>
-      <collision>
-        <origin xyz="0 0 0" rpy="0 0 0" />
-        <geometry>
-          <mesh filename="package://rr_robot_description/include/chassis/meshes/ToolHolder/collision.STL" />
-        </geometry>
-      </collision>
-    </link>
-    <joint name="th2_joint" type="fixed">
-      <origin
-        xyz="0.67894 0.175 0.12783"
-        rpy="-1.0611E-15 7.6478E-16 1.5708" />
-      <parent link="${name}" />
-      <child link="th2" />
-    </joint>
-    <link name="th3" >
-      <inertial>
-        <mass value="0.1911" />
-        <origin xyz="0 0 0" rpy="0 0 0" />
-        <inertia ixx="0.01880039566" ixy="-0.00288516792" ixz="0.00164510501" iyy="0.00519681040" iyz="-0.00798447007" izz="0.01485438661"/>
-      </inertial>
-      <visual>
-        <origin xyz="0 0 0" rpy="0 0 0" />
-        <geometry>
-          <mesh filename="package://rr_robot_description/include/chassis/meshes/ToolHolder/visual.STL" />
-        </geometry>
-        <material name="black">
-          <color rgba="0.2 0.2 0.2 1" />
-        </material>
-      </visual>
-      <collision>
-        <origin xyz="0 0 0" rpy="0 0 0" />
-        <geometry>
-          <mesh filename="package://rr_robot_description/include/chassis/meshes/ToolHolder/collision.STL" />
-        </geometry>
-      </collision>
-    </link>
-    <joint name="th3_joint" type="fixed">
-      <origin
-        xyz="0.67894 0 0.12783"
-        rpy="-1.0611E-15 7.6478E-16 1.5708" />
-      <parent link="${name}" />
-      <child link="th3" />
-    </joint>
-    <link name="th4" >
-      <inertial>
-        <mass value="0.1911" />
-        <origin xyz="0 0 0" rpy="0 0 0" />
-        <inertia ixx="0.01880039566" ixy="-0.00288516792" ixz="0.00164510501" iyy="0.00519681040" iyz="-0.00798447007" izz="0.01485438661"/>
-      </inertial>
-      <visual>
-        <origin xyz="0 0 0" rpy="0 0 0" />
-        <geometry>
-          <mesh filename="package://rr_robot_description/include/chassis/meshes/ToolHolder/visual.STL" />
-        </geometry>
-        <material name="black">
-          <color rgba="0.2 0.2 0.2 1" />
-        </material>
-      </visual>
-      <collision>
-        <origin xyz="0 0 0" rpy="0 0 0" />
-        <geometry>
-          <mesh filename="package://rr_robot_description/include/chassis/meshes/ToolHolder/collision.STL" />
-        </geometry>
-      </collision>
-    </link>
-    <joint name="th4_joint" type="fixed">
-      <origin
-        xyz="0.67894 -0.175 0.12783"
-        rpy="-1.0611E-15 7.6478E-16 1.5708" />
-      <parent
-        link="${name}" />
-      <child
-        link="th4" />
-    </joint>
-    <link name="th5" >
-      <inertial>
-        <mass value="0.1911" />
-        <origin xyz="0 0 0" rpy="0 0 0" />
-        <inertia ixx="0.01880039566" ixy="-0.00288516792" ixz="0.00164510501" iyy="0.00519681040" iyz="-0.00798447007" izz="0.01485438661"/>
-      </inertial>
-      <visual>
-        <origin xyz="0 0 0" rpy="0 0 0" />
-        <geometry>
-          <mesh filename="package://rr_robot_description/include/chassis/meshes/ToolHolder/visual.STL" />
-        </geometry>
-        <material name="black">
-          <color rgba="0.2 0.2 0.2 1" />
-        </material>
-      </visual>
-      <collision>
-        <origin xyz="0 0 0" rpy="0 0 0" />
-        <geometry>
-          <mesh filename="package://rr_robot_description/include/chassis/meshes/ToolHolder/collision.STL" />
-        </geometry>
-      </collision>
-    </link>
-    <joint name="th5_joint" type="fixed">
-      <origin
-        xyz="0.40394 0.175 0.12783"
-        rpy="-1.0611E-15 7.6478E-16 1.5708" />
-      <parent link="${name}" />
-      <child link="th5" />
-    </joint>
-    <link name="th6" >
-      <inertial>
-        <mass value="0.1911" />
-        <origin xyz="0 0 0" rpy="0 0 0" />
-        <inertia ixx="0.01880039566" ixy="-0.00288516792" ixz="0.00164510501" iyy="0.00519681040" iyz="-0.00798447007" izz="0.01485438661"/>
-      </inertial>
-      <visual>
-        <origin xyz="0 0 0" rpy="0 0 0" />
-        <geometry>
-          <mesh filename="package://rr_robot_description/include/chassis/meshes/ToolHolder/visual.STL" />
-        </geometry>
-        <material name="black">
-          <color rgba="0.2 0.2 0.2 1" />
-        </material>
-      </visual>
-      <collision>
-        <origin xyz="0 0 0" rpy="0 0 0" />
-        <geometry>
-          <mesh filename="package://rr_robot_description/include/chassis/meshes/ToolHolder/collision.STL" />
-        </geometry>
-      </collision>
-    </link>
-    <joint name="th6_joint" type="fixed">
-      <origin
-        xyz="0.40394 0 0.12783"
-        rpy="-1.0611E-15 7.6478E-16 1.5708" />
-      <parent link="${name}" />
-      <child link="th6" />
-    </joint>
-    <link name="th7" >
-      <inertial>
-        <mass value="0.1911" />
-        <origin xyz="0 0 0" rpy="0 0 0" />
-        <inertia ixx="0.01880039566" ixy="-0.00288516792" ixz="0.00164510501" iyy="0.00519681040" iyz="-0.00798447007" izz="0.01485438661"/>
-      </inertial>
-      <visual>
-        <origin xyz="0 0 0" rpy="0 0 0" />
-        <geometry>
-          <mesh filename="package://rr_robot_description/include/chassis/meshes/ToolHolder/visual.STL" />
-        </geometry>
-        <material name="black">
-          <color rgba="0.2 0.2 0.2 1" />
-        </material>
-      </visual>
-      <collision>
-        <origin xyz="0 0 0" rpy="0 0 0" />
-        <geometry>
-          <mesh filename="package://rr_robot_description/include/chassis/meshes/ToolHolder/collision.STL" />
-        </geometry>
-      </collision>
-    </link>
-    <joint name="th7_joint" type="fixed">
-      <origin
-        xyz="0.40394 -0.175 0.12783"
-        rpy="-1.0611E-15 7.6478E-16 1.5708" />
-      <parent link="${name}" />
-      <child link="th7" />
-    </joint>
+    <xacro:include filename="$(find rr_robot_description)/include/chassis/urdf/tool_holder.xacro"/>
+    <xacro:tool_holder_macro name="th0" parent="${name}" x_offset="0.95394" y_offset="0.0875" z_offset="0.12783" yaw="1.5708"/>
+    <xacro:tool_holder_macro name="th1" parent="${name}" x_offset="0.95394" y_offset="-0.0875" z_offset="0.12783" yaw="1.5708"/>
+    <xacro:tool_holder_macro name="th2" parent="${name}" x_offset="0.67894" y_offset="0.175" z_offset="0.12783" yaw="1.5708"/>
+    <xacro:tool_holder_macro name="th3" parent="${name}" x_offset="0.67894" y_offset="0." z_offset="0.12783" yaw="1.5708"/>
+    <xacro:tool_holder_macro name="th4" parent="${name}" x_offset="0.67894" y_offset="-0.175" z_offset="0.12783" yaw="1.5708"/>
+    <xacro:tool_holder_macro name="th5" parent="${name}" x_offset="0.40394" y_offset="0.175" z_offset="0.12783" yaw="1.5708"/>
+    <xacro:tool_holder_macro name="th6" parent="${name}" x_offset="0.40394" y_offset="0." z_offset="0.12783" yaw="1.5708"/>
+    <xacro:tool_holder_macro name="th7" parent="${name}" x_offset="0.40394" y_offset="-0.175" z_offset="0.12783" yaw="1.5708"/>
   </xacro:macro>
 </robot>
