Commit message: cmd_vel controller + rope drive joints

File: src/rr_robot_description/include/chassis/urdf/chassis.xacro (robot description, xacro)
@@ -62,5 +62,5 @@
       <inertial>
         <mass value="2.206" />
-        <origin xyz="0.01032 0 0" rpy="0 0 0" />
+        <origin xyz="0 0 0" rpy="0 0 0" />
         <inertia ixx="0.00699387" ixy="0" ixz="0" iyy="0.0044146" iyz="0" izz="0.0044146"/>
       </inertial>
@@ -81,5 +81,5 @@
       </collision>
     </link>
-    <joint name="rope_drive_le_joint" type="fixed">
+    <joint name="rope_drive_le_joint" type="continuous">
       <origin xyz="0.92999 0.24067 -0.0269" rpy="-0.09857 0.09857 -1.64405" />
       <axis rpy="0 0 0" xyz="1 0 0" />
@@ -111,5 +111,5 @@
       </collision>
     </link>
-    <joint name="rope_drive_te_joint" type="fixed">
+    <joint name="rope_drive_te_joint" type="continuous">
       <origin xyz="0.92999 -0.24067 -0.0269" rpy="0.09857 0.09857 1.64405" />
       <axis rpy="0 0 0" xyz="1 0 0" />

Commit message: Cmd_vel controller working

File: src/rr_robot_description/include/chassis/urdf/chassis.xacro (robot description, xacro)
@@ -113,5 +113,5 @@
     <joint name="rope_drive_te_joint" type="continuous">
       <origin xyz="0.92999 -0.24067 -0.0269" rpy="0.09857 0.09857 1.64405" />
-      <axis rpy="0 0 0" xyz="1 0 0" />
+      <axis rpy="0 0 0" xyz="-1 0 0" />
       <limit effort="10000" velocity="1000" />
       <joint_properties damping="1.0" friction="1.0" />

File: src/rr_robot_description/urdf/robot.urdf.xacro (robot description, xacro)
@@ -100,8 +100,4 @@
   <!-- ******************************** Tranmissions ******************************** -->
   <xacro:include filename="$(find rr_robot_description)/urdf/transmissions.xacro" />
-  <!--***************************** Rope for winch plugin *****************************-->
-  <xacro:include filename="$(find rr_robot_description)/urdf/rope.xacro" />
-  <xacro:rope_macro winch_name_no_postfix="rope_drive"
-                    rope_l="50"/>
   <!-- *********************************** Gazebo *********************************** -->
   <xacro:include filename="$(find rr_robot_description)/urdf/robot.gazebo" />

File: src/rr_robot_description/urdf/transmissions.xacro (robot description, xacro)
@@ -46,9 +46,3 @@
     <xacro:EffortJointMacro joint_name="bot_wheel_joint_le"/>
     <xacro:EffortJointMacro joint_name="bot_wheel_joint_te"/>
-    <xacro:EffortJointMacro joint_name="rope_yaw_te_joint"/>
-    <xacro:EffortJointMacro joint_name="rope_yaw_le_joint"/>
-    <xacro:EffortJointMacro joint_name="rope_pitch_te_joint"/>
-    <xacro:EffortJointMacro joint_name="rope_pitch_le_joint"/>
-    <xacro:EffortJointMacro joint_name="rope_springed_joint_te"/>
-    <xacro:EffortJointMacro joint_name="rope_springed_joint_le"/>
 </robot>

File: src/rr_robot_description/urdf/wheel_assembly/bot_wheel.xacro (robot description, xacro)
@@ -33,5 +33,5 @@
                 <parent link="${parent}" />
                 <child link="bot_wheel_mount_${postfix}"/>
-                <dynamics damping="1" />
+                <dynamics damping="30" />
             </joint>
         <!-- Wheel -->

File: src/rr_robot_description/urdf/wheel_assembly/top_wheel.xacro (robot description, xacro)
@@ -35,5 +35,5 @@
               <parent link="${parent}" />
               <child link="top_wheel_mount_${postfix}"/>
-              <dynamics damping="1" />
+              <dynamics damping="30" />
           </joint>
           <link name="yaw_link_${postfix}">

Commit message: Updated vacuum to correct normal force on chassis

File: src/rr_robot_description/include/chassis/urdf/chassis.xacro (robot description, xacro)
@@ -17,10 +17,10 @@
         </material>
       </visual>
-      <collision>
+      <!-- <collision>
         <origin xyz="0 0 0" rpy="0 0 0" />
         <geometry>
           <mesh filename="package://rr_robot_description/include/chassis/meshes/Chassis/collision.STL" />
         </geometry>
-      </collision>
+      </collision> -->
     </link>
     <joint name="${parent_link}_to_${name}" type="fixed">

File: src/rr_robot_description/urdf/wheel_assembly/bot_wheel.xacro (robot description, xacro)
@@ -4,6 +4,6 @@
     the range of motion is small -->
 <robot xmlns:xacro="http://ros.org/wiki/xacro" name="bot_wheel">
-    <xacro:property name="range" value="0.174533" />
     <xacro:macro name="bot_wheels_macro" params="parent x z wspan">
+        <xacro:property name="range" value="0.174533" />
         <xacro:macro name="make_bot_wheel" params="te='true'">
             <xacro:if value="${te}">
@@ -33,5 +33,5 @@
                 <parent link="${parent}" />
                 <child link="bot_wheel_mount_${postfix}"/>
-                <dynamics damping="30" />
+                <dynamics damping="30" friction="1" />
             </joint>
         <!-- Wheel -->

File: src/rr_robot_description/urdf/wheel_assembly/top_wheel.xacro (robot description, xacro)
@@ -4,6 +4,6 @@
     the range of motion is small -->
 <robot xmlns:xacro="http://ros.org/wiki/xacro" name="top_wheels">
+    <xacro:macro name="top_wheels_macro" params="parent x z wspan">
     <xacro:property name="range" value="0.174533" />
-    <xacro:macro name="top_wheels_macro" params="parent x z wspan">
       <!-- Macro for making a single wheel-->
       <xacro:macro name="make_wheel" params="te='true'">
@@ -35,5 +35,5 @@
               <parent link="${parent}" />
               <child link="top_wheel_mount_${postfix}"/>
-              <dynamics damping="30" />
+              <dynamics damping="30" friction="1"/>
           </joint>
           <link name="yaw_link_${postfix}">
@@ -48,8 +48,7 @@
               <axis xyz="0 0 1" />
               <limit lower="-0.20" upper="0.20" effort="1000000" velocity="1000" />
-              <joint_properties damping="1.0" friction="1.0" />
               <parent link="top_wheel_mount_${postfix}" />
               <child link="yaw_link_${postfix}" />
-              <dynamics damping="1" />
+              <dynamics damping="1"/>
           </joint>
           <link name="top_wheel_${postfix}">

Commit message: prismatic joint for vacuum sheet (fixed for now)

File: src/rr_robot_description/include/chassis/urdf/chassis.xacro (robot description, xacro)
@@ -136,7 +136,8 @@
       </visual>
       <!-- Collision of vacuum sheet is neglected -->
-      <!--<collision>
+      <!-- <collision>
         <origin xyz="0 0 0" rpy="0 0 0" />
         <geometry>
+          <box size="0.5 0.2 0.1"/>
           <mesh filename="package://rr_robot_description/include/chassis/meshes/VacuumSheet/collision.STL" />
         </geometry>
@@ -144,5 +145,8 @@
     </link>
     <joint name="vacuum_sheet_joint" type="fixed">
+      <dynamics damping="10" friction="10"/>
       <origin xyz="0.55919 0. -0.145" rpy="0. 0. 1.5708" />
+      <limit lower="0" upper="1" effort="10000" velocity="1000"/>
+      <axis xyz="0 0 1"/>
       <parent link="${name}" />
       <child link="vacuum_sheet" />
