Commit message: winch plugin working + yaw controller working

File: src/rr_robot_description/urdf/wheel_assembly/top_wheel.xacro (robot description, xacro)
@@ -32,5 +32,5 @@
               <origin xyz="${x-0.10581} ${y-yaw_arm} ${z-0.01217}" rpy="0 0 0" />
               <axis xyz="0 1 0" />
-              <limit lower="${-range}" upper="${range}" effort="1000" velocity="1000"/>
+              <limit lower="${-range}" upper="${range}" effort="10000000" velocity="100000"/>
               <parent link="${parent}" />
               <child link="top_wheel_mount_${postfix}"/>
@@ -47,5 +47,5 @@
               <origin xyz="0.10581 0 0.01217" rpy="0. 0. 1.5708" />
               <axis xyz="0 0 1" />
-              <limit lower="-0.20" upper="0.20" effort="10000" velocity="1000" />
+              <limit lower="-0.20" upper="0.20" effort="1000000" velocity="1000" />
               <joint_properties damping="1.0" friction="1.0" />
               <parent link="top_wheel_mount_${postfix}" />

Commit message: Collision geometry changed

File: src/rr_robot_description/urdf/wheel_assembly/top_wheel.xacro (robot description, xacro)
@@ -32,5 +32,5 @@
         <parent link="${parent}" />
         <child link="top_wheel_mount_${postfix}" />
-        <dynamics damping="1" friction="1" />
+        <dynamics damping="1" friction="10" />
       </joint>
       <link name="yaw_link_${postfix}">
@@ -68,8 +68,9 @@
         </visual>
         <collision>
-          <origin xyz="0 0 0" rpy="0 0 0" />
+          <origin xyz="0 0 0" rpy="0 1.57079633 0" />
           <geometry>
-            <mesh
-              filename="package://rr_robot_description/include/chassis/meshes/BottomWheels/collision.STL" />
+            <cylinder radius="0.05" length="0.02"/>
+            <!-- <mesh
+              filename="package://rr_robot_description/include/chassis/meshes/BottomWheels/collision.STL" /> -->
           </geometry>
         </collision>
@@ -80,5 +81,5 @@
         <parent link="yaw_link_${postfix}" />
         <child link="top_wheel_${postfix}" />
-        <dynamics damping="1" />
+        <dynamics damping="1" friction="10"/>
       </joint>
     </xacro:macro>

Commit message: decreased max allowed eff and vel

File: src/rr_robot_description/urdf/wheel_assembly/top_wheel.xacro (robot description, xacro)
@@ -29,5 +29,5 @@
         <origin xyz="${x-0.10581} ${y-yaw_arm} ${z-0.01217}" rpy="0 0 0" />
         <axis xyz="0 1 0" />
-        <limit lower="${-range}" upper="${range}" effort="10000000" velocity="100000" />
+        <limit lower="${-range}" upper="${range}" effort="10000" velocity="100" />
         <parent link="${parent}" />
         <child link="top_wheel_mount_${postfix}" />
@@ -45,5 +45,5 @@
         <origin xyz="0.10581 0 0.01217" rpy="0. 0. 1.5708" />
         <axis xyz="0 0 1" />
-        <limit lower="-0.20" upper="0.20" effort="1000000" velocity="1000" />
+        <limit lower="-0.20" upper="0.20" effort="500" velocity="5" />
         <parent link="top_wheel_mount_${postfix}" />
         <child link="yaw_link_${postfix}" />

Commit message: yaw angle limit bug fixed

File: src/rr_robot_description/urdf/wheel_assembly/top_wheel.xacro (robot description, xacro)
@@ -45,5 +45,5 @@
         <origin xyz="0.09941 0 0.02003" rpy="0. 0. 1.5708" />
         <axis xyz="0 0 1" />
-        <limit lower="0" upper="0.20" effort="500" velocity="5" />
+        <limit lower="-0.2" upper="0.2" effort="500" velocity="5" />
         <parent link="top_wheel_mount_${postfix}" />
         <child link="yaw_link_${postfix}" />
