Commit message: Changed solver settings and colission geometry

File: src/rr_robot_description/urdf/wheel_assembly/bot_wheel.xacro (robot description, xacro)
@@ -30,5 +30,5 @@
                 <parent link="${parent}" />
                 <child link="bot_wheel_mount_${postfix}" />
-                <dynamics damping="1" friction="1" />
+                <dynamics damping="1" friction="10" />
             </joint>
             <!-- Wheel -->
@@ -50,8 +50,9 @@
                 </visual>
                 <collision>
-                    <origin xyz="0 0 0" rpy="0 0 0" />
+                    <origin xyz="0 0 0" rpy="0 1.57079633 0" />
                     <geometry>
-                        <mesh
-                            filename="package://rr_robot_description/include/chassis/meshes/BottomWheels/collision.STL" />
+                        <cylinder radius="0.05" length="0.02"/>
+                        <!-- <mesh
+                            filename="package://rr_robot_description/include/chassis/meshes/BottomWheels/collision.STL" /> -->
                     </geometry>
                 </collision>
@@ -62,5 +63,5 @@
                 <parent link="bot_wheel_mount_${postfix}" />
                 <child link="bot_wheel_${postfix}" />
-                <dynamics damping="1" />
+                <dynamics damping="1" friction="10"/>
             </joint>
         </xacro:macro>

Commit message: Damping added and friction lowered on wheels

File: src/rr_robot_description/urdf/wheel_assembly/bot_wheel.xacro (robot description, xacro)
@@ -48,5 +48,5 @@
                     </material>
                 </visual>
-                <collision>
+                <collision name="bot_wheel_${postfix}_collision">
                     <origin xyz="0 0 0" rpy="0 1.57079633 0" />
                     <geometry>
@@ -62,5 +62,5 @@
                 <parent link="bot_wheel_mount_${postfix}" />
                 <child link="bot_wheel_${postfix}" />
-                <dynamics damping="1" friction="10"/>
+                <dynamics damping="0" friction="0.1"/>
             </joint>
         </xacro:macro>

File: src/rr_robot_description/urdf/wheel_assembly/top_wheel.xacro (robot description, xacro)
@@ -81,5 +81,5 @@
         <parent link="yaw_link_${postfix}" />
         <child link="top_wheel_${postfix}" />
-        <dynamics damping="1" friction="10"/>
+        <dynamics damping="0" friction="0.1"/>
       </joint>
     </xacro:macro>
